Commit message: Gazebo now works a little better. Small fixes in driver/camera.
Also, I added 'Body' group in srdf files to be able to control all joints at once in MoveIt!

File: nao_dcm_common/nao_dcm_description/urdf/nao_dcm_H21_structure.xacro (robot description, xacro)
@@ -17,4 +17,11 @@
         </inertial>
     </link>
+    <!-- IMU -->
+    <joint name="torso-imu" type="fixed">
+        <parent link="torso"/>
+        <child link="imu"/>
+        <origin xyz="-0.008 0.00606 0.027" rpy="0 0 0"/>
+    </joint>
+    <link name="imu"/>
     <!-- SONARS -->
     <!-- Nao has different sonar transmitter and receiver. The correct way is to take the intersection of the 2 cones -->

File: nao_dcm_common/nao_dcm_description/urdf/nao_dcm_H25_structure.xacro (robot description, xacro)
@@ -17,4 +17,11 @@
         </inertial>
     </link>
+    <!-- IMU -->
+    <joint name="torso-imu" type="fixed">
+        <parent link="torso"/>
+        <child link="imu"/>
+        <origin xyz="-0.008 0.00606 0.027" rpy="0 0 0"/>
+    </joint>
+    <link name="imu"/>
     <!-- SONARS -->
     <!-- Nao has different sonar transmitter and receiver. The correct way is to take the intersection of the 2 cones -->
@@ -177,5 +184,11 @@
         <limit effort="0.49" lower="0.0" upper="1.0" velocity="3.0"/>
     </joint>
-    <link name="l_gripper"/>
+    <link name="l_gripper">
+        <inertial> <!-- dummy values for gazebo -->
+            <mass value="1e-5" />
+            <origin xyz="0 0 0"/>
+            <inertia ixx="1e-9" ixy="0" ixz="0" iyy="1e-9" iyz="0" izz="1e-9" />
+        </inertial>
+    </link>
     <joint name="RWristYaw" type="revolute">
         <parent link="RElbowDummy"/>
@@ -200,5 +213,11 @@
         <limit effort="0.49" lower="0.0" upper="1.0" velocity="3.0"/>
     </joint>
-    <link name="r_gripper"/>
+    <link name="r_gripper">
+        <inertial> <!-- dummy values for gazebo -->
+            <mass value="1e-5" />
+            <origin xyz="0 0 0"/>
+            <inertia ixx="1e-9" ixy="0" ixz="0" iyy="1e-9" iyz="0" izz="1e-9" />
+        </inertial>
+    </link>
     <!-- JOINTS THAT ARE NOT IDENTICAL TO 2 ENDS -->
     <joint name="LShoulderRoll" type="revolute">

File: nao_dcm_common/nao_dcm_description/urdf/nao_dcm_gazebo.xacro (robot description, xacro)
@@ -1,9 +1,17 @@
 <?xml version="1.0"?>
 <robot xmlns:xacro="http://www.ros.org/wiki/xacro">
-    <!-- GAZEBO ROS CONTROL PLUGIN -->
+    <!-- GAZEBO ROS CONTROL AND IMU PLUGIN -->
     <gazebo>
         <plugin filename="libgazebo_ros_control.so" name="gazebo_ros_control">
             <robotNamespace>/nao_dcm</robotNamespace>
             <robotSimType>gazebo_ros_control/DefaultRobotHWSim</robotSimType>
+        </plugin>
+        <plugin name="gazebo_ros_imu_controller" filename="libgazebo_ros_imu.so">
+            <robotNamespace>/nao_dcm</robotNamespace>
+            <topicName>imu_data</topicName>
+            <bodyName>imu</bodyName>
+            <gaussianNoise>2.89e-08</gaussianNoise>
+            <xyzOffsets>0 0 0</xyzOffsets>
+            <rpyOffsets>0 0 0</rpyOffsets>
         </plugin>
     </gazebo>
@@ -228,5 +236,5 @@
                 <alwaysOn>true</alwaysOn>
                 <updateRate>0.0</updateRate>
-                <cameraName>nao_robot/CameraTop</cameraName>
+                <cameraName>nao_dcm/CameraTop</cameraName>
                 <imageTopicName>image_raw</imageTopicName>
                 <cameraInfoTopicName>camera_info</cameraInfoTopicName>
@@ -264,5 +272,5 @@
                 <alwaysOn>true</alwaysOn>
                 <updateRate>0.0</updateRate>
-                <cameraName>nao_robot/CameraBottom</cameraName>
+                <cameraName>nao_dcm/CameraBottom</cameraName>
                 <imageTopicName>image_raw</imageTopicName>
                 <cameraInfoTopicName>camera_info</cameraInfoTopicName>

Commit message: Fixed joint efforts for Gazebo and parameters..

File: nao_dcm_common/nao_dcm_description/urdf/nao_dcm_H21_structure.xacro (robot description, xacro)
@@ -54,5 +54,5 @@
         <parent link="torso"/>
         <child link="neck"/>
-        <limit effort="0.62" lower="-2.0857" upper="2.0857" velocity="3.0"/>
+        <limit effort="5" lower="-2.0857" upper="2.0857" velocity="3.0"/>
         <origin rpy="0 0 0" xyz="0 0 0.1265"/>
         <axis xyz="0 0 1"/>
@@ -71,5 +71,5 @@
         <parent link="neck"/>
         <child link="gaze"/>
-        <limit effort="0.62" lower="-0.6720" upper="0.5149" velocity="3.0"/>
+        <limit effort="5" lower="-0.6720" upper="0.5149" velocity="3.0"/>
         <origin rpy="0 0 0" xyz="0 0 0"/>
         <axis xyz="0 1 0"/>
@@ -122,5 +122,5 @@
             <parent link="torso"/>
             <child link="${side}Shoulder"/>
-            <limit effort="0.62" lower="-2.0857" upper="2.0857" velocity="3.0"/>
+            <limit effort="5" lower="-2.0857" upper="2.0857" velocity="3.0"/>
             <origin rpy="0 0 0" xyz="0 ${reflect*0.098} 0.1"/>
             <axis xyz="0 1 0"/>
@@ -137,5 +137,5 @@
             <parent link="${side}ShoulderDummy"/>
             <child link="${side}Elbow"/>
-            <limit effort="0.62" lower="-2.0857" upper="2.0857" velocity="3.0"/>
+            <limit effort="5" lower="-2.0857" upper="2.0857" velocity="3.0"/>
             <origin rpy="0 0 0" xyz="0.105 ${reflect*0.015} 0"/>
             <axis xyz="1 0 0"/>
@@ -194,5 +194,5 @@
         <parent link="LShoulder"/>
         <child link="LShoulderDummy"/>
-        <limit effort="0.62" lower="-0.3142" upper="1.3265" velocity="3.0"/>
+        <limit effort="5" lower="-0.3142" upper="1.3265" velocity="3.0"/>
         <origin rpy="0 0 0" xyz="0 0 0"/>
         <axis xyz="0 0 1"/>
@@ -201,5 +201,5 @@
         <parent link="RShoulder"/>
         <child link="RShoulderDummy"/>
-        <limit effort="0.62" lower="-1.3265" upper="0.3142" velocity="3.0"/>
+        <limit effort="5" lower="-1.3265" upper="0.3142" velocity="3.0"/>
         <origin rpy="0 0 0" xyz="0 0 0"/>
         <axis xyz="0 0 1"/>
@@ -208,5 +208,5 @@
         <parent link="LElbow"/>
         <child link="LElbowDummy"/>
-        <limit effort="0.62" lower="-1.5446" upper="-0.0349" velocity="3.0"/>
+        <limit effort="5" lower="-1.5446" upper="-0.0349" velocity="3.0"/>
         <origin rpy="0 0 0" xyz="0 0 0"/>
         <axis xyz="0 0 1"/>
@@ -215,5 +215,5 @@
         <parent link="RElbow"/>
         <child link="RElbowDummy"/>
-        <limit effort="0.62" lower="0.0349" upper="1.5446" velocity="3.0"/>
+        <limit effort="5" lower="0.0349" upper="1.5446" velocity="3.0"/>
         <origin rpy="0 0 0" xyz="0 0 0"/>
         <axis xyz="0 0 1"/>
@@ -224,5 +224,5 @@
         <parent link="base_link"/>
         <child link="LHipYaw"/>
-        <limit effort="1.61" lower="-1.145303" upper="0.740810" velocity="3.0"/>
+        <limit effort="5" lower="-1.145303" upper="0.740810" velocity="3.0"/>
         <origin rpy="0 0 0" xyz="0 0.05 -0.085"/>
         <axis xyz="0 0.707106 -0.707106"/>
@@ -240,5 +240,5 @@
         <parent link="LHipYaw"/>
         <child link="LHip"/>
-        <limit effort="1.61" lower="-0.379472" upper="0.790477" velocity="3.0"/>
+        <limit effort="5" lower="-0.379472" upper="0.790477" velocity="3.0"/>
         <origin rpy="0 0 0" xyz="0 0 0"/>
         <axis xyz="1 0 0"/>
@@ -256,5 +256,5 @@
         <parent link="LHip"/>
         <child link="LHipDummy"/>
-        <limit effort="1.61" lower="-1.535889" upper="0.484090" velocity="3.0"/>
+        <limit effort="5" lower="-1.535889" upper="0.484090" velocity="3.0"/>
         <origin rpy="0 0 0" xyz="0 0 0"/>
         <axis xyz="0 1 0"/>
@@ -272,5 +272,5 @@
         <parent link="LHipDummy"/>
         <child link="LKnee"/>
-        <limit effort="1.61" lower="-0.092346" upper="2.112528" velocity="3.0"/>
+        <limit effort="5" lower="-0.092346" upper="2.112528" velocity="3.0"/>
         <origin rpy="0 0 0" xyz="0 0 -0.1"/>
         <axis xyz="0 1 0"/>
@@ -288,5 +288,5 @@
         <parent link="LKnee"/>
         <child link="l_ankle"/>
-        <limit effort="1.61" lower="-1.189516" upper="0.922747" velocity="3.0"/>
+        <limit effort="5" lower="-1.189516" upper="0.922747" velocity="3.0"/>
         <origin rpy="0 0 0" xyz="0 0 -0.1029"/>
         <axis xyz="0 1 0"/>
@@ -304,5 +304,5 @@
         <parent link="l_ankle"/>
         <child link="l_sole"/>
-        <limit effort="1.61" lower="-0.397880" upper="0.769001" velocity="3.0"/>
+        <limit effort="5" lower="-0.397880" upper="0.769001" velocity="3.0"/>
         <origin rpy="0 0 0" xyz="0 0 0"/>
         <axis xyz="1 0 0"/>
@@ -321,5 +321,5 @@
         <parent link="base_link"/>
         <child link="RHipYaw"/>
-        <limit effort="1.61" lower="-1.145303" upper="0.740810" velocity="3.0"/>
+        <limit effort="5" lower="-1.145303" upper="0.740810" velocity="3.0"/>
         <origin rpy="0 0 0" xyz="0 -0.05 -0.085"/>
         <axis xyz="0 0.707106 0.707106"/>
@@ -338,5 +338,5 @@
         <parent link="RHipYaw"/>
         <child link="RHip"/>
-        <limit effort="1.61" lower="-0.790477" upper="0.379472" velocity="3.0"/>
+        <limit effort="5" lower="-0.790477" upper="0.379472" velocity="3.0"/>
         <origin rpy="0 0 0" xyz="0 0 0"/>
         <axis xyz="1 0 0"/>
@@ -354,5 +354,5 @@
         <parent link="RHip"/>
         <child link="RHipDummy"/>
-        <limit effort="1.61" lower="-1.535889" upper="0.484090" velocity="3.0"/>
+        <limit effort="5" lower="-1.535889" upper="0.484090" velocity="3.0"/>
         <origin rpy="0 0 0" xyz="0 0 0"/>
         <axis xyz="0 1 0"/>
@@ -370,5 +370,5 @@
         <parent link="RHipDummy"/>
         <child link="RKnee"/>
-        <limit effort="1.61" lower="-0.103083" upper="2.120198" velocity="3.0"/>
+        <limit effort="5" lower="-0.103083" upper="2.120198" velocity="3.0"/>
         <origin rpy="0 0 0" xyz="0 0 -0.1"/>
         <axis xyz="0 1 0"/>
@@ -386,5 +386,5 @@
         <parent link="RKnee"/>
         <child link="r_ankle"/>
-        <limit effort="1.61" lower="-1.186448" upper="0.932056" velocity="3.0"/>
+        <limit effort="5" lower="-1.186448" upper="0.932056" velocity="3.0"/>
         <origin rpy="0 0 0" xyz="0 0 -0.1029"/>
         <axis xyz="0 1 0"/>
@@ -402,5 +402,5 @@
         <parent link="r_ankle"/>
         <child link="r_sole"/>
-        <limit effort="1.61" lower="-0.768992" upper="0.397935" velocity="3.0"/>
+        <limit effort="5" lower="-0.768992" upper="0.397935" velocity="3.0"/>
         <origin rpy="0 0 0" xyz="0 0 0"/>
         <axis xyz="1 0 0"/>

File: nao_dcm_common/nao_dcm_description/urdf/nao_dcm_H25_structure.xacro (robot description, xacro)
@@ -54,5 +54,5 @@
         <parent link="torso"/>
         <child link="neck"/>
-        <limit effort="0.62" lower="-2.0857" upper="2.0857" velocity="3.0"/>
+        <limit effort="5" lower="-2.0857" upper="2.0857" velocity="3.0"/>
         <origin rpy="0 0 0" xyz="0 0 0.1265"/>
         <axis xyz="0 0 1"/>
@@ -71,5 +71,5 @@
         <parent link="neck"/>
         <child link="gaze"/>
-        <limit effort="0.62" lower="-0.6720" upper="0.5149" velocity="3.0"/>
+        <limit effort="5" lower="-0.6720" upper="0.5149" velocity="3.0"/>
         <origin rpy="0 0 0" xyz="0 0 0"/>
         <axis xyz="0 1 0"/>
@@ -122,5 +122,5 @@
             <parent link="torso"/>
             <child link="${side}Shoulder"/>
-            <limit effort="0.62" lower="-2.0857" upper="2.0857" velocity="3.0"/>
+            <limit effort="5" lower="-2.0857" upper="2.0857" velocity="3.0"/>
             <origin rpy="0 0 0" xyz="0 ${reflect*0.098} 0.1"/>
             <axis xyz="0 1 0"/>
@@ -137,5 +137,5 @@
             <parent link="${side}ShoulderDummy"/>
             <child link="${side}Elbow"/>
-            <limit effort="0.62" lower="-2.0857" upper="2.0857" velocity="3.0"/>
+            <limit effort="5" lower="-2.0857" upper="2.0857" velocity="3.0"/>
             <origin rpy="0 0 0" xyz="0.105 ${reflect*0.015} 0"/>
             <axis xyz="1 0 0"/>
@@ -224,5 +224,5 @@
         <parent link="LShoulder"/>
         <child link="LShoulderDummy"/>
-        <limit effort="0.62" lower="-0.3142" upper="1.3265" velocity="3.0"/>
+        <limit effort="5" lower="-0.3142" upper="1.3265" velocity="3.0"/>
         <origin rpy="0 0 0" xyz="0 0 0"/>
         <axis xyz="0 0 1"/>
@@ -231,5 +231,5 @@
         <parent link="RShoulder"/>
         <child link="RShoulderDummy"/>
-        <limit effort="0.62" lower="-1.3265" upper="0.3142" velocity="3.0"/>
+        <limit effort="5" lower="-1.3265" upper="0.3142" velocity="3.0"/>
         <origin rpy="0 0 0" xyz="0 0 0"/>
         <axis xyz="0 0 1"/>
@@ -238,5 +238,5 @@
         <parent link="LElbow"/>
         <child link="LElbowDummy"/>
-        <limit effort="0.62" lower="-1.5446" upper="-0.0349" velocity="3.0"/>
+        <limit effort="5" lower="-1.5446" upper="-0.0349" velocity="3.0"/>
         <origin rpy="0 0 0" xyz="0 0 0"/>
         <axis xyz="0 0 1"/>
@@ -245,5 +245,5 @@
         <parent link="RElbow"/>
         <child link="RElbowDummy"/>
-        <limit effort="0.62" lower="0.0349" upper="1.5446" velocity="3.0"/>
+        <limit effort="5" lower="0.0349" upper="1.5446" velocity="3.0"/>
         <origin rpy="0 0 0" xyz="0 0 0"/>
         <axis xyz="0 0 1"/>
