Commit message: Converted nao_meshes to collada for Gazebo compatibility..

File: nao_dcm_common/nao_dcm_description/urdf/nao_dcm_visuals_collisions.xacro (robot description, xacro)
@@ -14,4 +14,7 @@
 		<color rgba="1 1 0 1"/>
     </material>
+    <material name="LightGrey">
+    	<color rgba="0.8 0.8 0.8 1.0"/>
+	</material>
     <!-- END OF MATERIALS -->
     <!-- XACRO MACROS FOR VISUALS AND COLLISIONS -->
@@ -34,14 +37,14 @@
 		<xacro:if value="${nao_meshes}">
 			<visual>
-				<origin xyz="0 0 0" rpy="0 -0 0"/>
-				<geometry>
-					<mesh filename="package://nao_meshes/meshes/V40/visual/Torso.obj"  scale="${scale} ${scale} ${scale}"/>
-				</geometry>
-				<material name="LightGrey"/>
-			</visual>
-			<collision>
-				<origin xyz="0 0 0" rpy="0 -0 0"/>
-				<geometry>
-					<mesh filename="package://nao_meshes/meshes/V40/collision/Torso.ply"  scale="${scale} ${scale} ${scale}"/>
+				<origin xyz="0 0 0" rpy="-${PI_2} -0 0"/>
+				<geometry>
+					<mesh filename="package://nao_meshes/meshes/V40/visual/Torso.dae"  scale="${scale} ${scale} ${scale}"/>
+				</geometry>
+				<material name="LightGrey"/>
+			</visual>
+			<collision>
+				<origin xyz="0 0 0" rpy="0 -0 0"/>
+				<geometry>
+					<mesh filename="package://nao_meshes/meshes/V40/collision/Torso.dae"  scale="${scale} ${scale} ${scale}"/>
 				</geometry>
 				<material name="LightGrey"/>
@@ -52,14 +55,14 @@
 		<xacro:if value="${nao_meshes}">
 			<visual>
-				<origin xyz="0 0 0" rpy="0 -0 0"/>
-				<geometry>
-					<mesh filename="package://nao_meshes/meshes/V40/visual/HeadYaw.obj"  scale="${scale} ${scale} ${scale}"/>
-				</geometry>
-				<material name="LightGrey"/>
-			</visual>
-			<collision>
-				<origin xyz="0 0 0" rpy="0 -0 0"/>
-				<geometry>
-					<mesh filename="package://nao_meshes/meshes/V40/collision/HeadYaw.ply"  scale="${scale} ${scale} ${scale}"/>
+				<origin xyz="0 0 0" rpy="-${PI_2} -0 0"/>
+				<geometry>
+					<mesh filename="package://nao_meshes/meshes/V40/visual/HeadYaw.dae"  scale="${scale} ${scale} ${scale}"/>
+				</geometry>
+				<material name="LightGrey"/>
+			</visual>
+			<collision>
+				<origin xyz="0 0 0" rpy="0 -0 0"/>
+				<geometry>
+					<mesh filename="package://nao_meshes/meshes/V40/collision/HeadYaw.dae"  scale="${scale} ${scale} ${scale}"/>
 				</geometry>
 				<material name="LightGrey"/>
@@ -85,14 +88,14 @@
 		<xacro:if value="${nao_meshes}">
 			<visual>
-				<origin xyz="0 0 0" rpy="0 -0 0"/>
-				<geometry>
-					<mesh filename="package://nao_meshes/meshes/V40/visual/HeadPitch.obj"  scale="${scale} ${scale} ${scale}"/>
-				</geometry>
-				<material name="LightGrey"/>
-			</visual>
-			<collision>
-				<origin xyz="0 0 0" rpy="0 -0 0"/>
-				<geometry>
-					<mesh filename="package://nao_meshes/meshes/V40/collision/HeadPitch.ply"  scale="${scale} ${scale} ${scale}"/>
+				<origin xyz="0 0 0" rpy="-${PI_2} -0 0"/>
+				<geometry>
+					<mesh filename="package://nao_meshes/meshes/V40/visual/HeadPitch.dae"  scale="${scale} ${scale} ${scale}"/>
+				</geometry>
+				<material name="LightGrey"/>
+			</visual>
+			<collision>
+				<origin xyz="0 0 0" rpy="0 -0 0"/>
+				<geometry>
+					<mesh filename="package://nao_meshes/meshes/V40/collision/HeadPitch.dae"  scale="${scale} ${scale} ${scale}"/>
 				</geometry>
 				<material name="LightGrey"/>
@@ -103,14 +106,14 @@
 		<xacro:if value="${nao_meshes}">
 			<visual>
-				<origin xyz="0 0 0" rpy="0 -0 0"/>
-				<geometry>
-					<mesh filename="package://nao_meshes/meshes/V40/visual/${side}ShoulderPitch.obj"  scale="${scale} ${scale} ${scale}"/>
-				</geometry>
-				<material name="LightGrey"/>
-			</visual>
-			<collision>
-				<origin xyz="0 0 0" rpy="0 -0 0"/>
-				<geometry>
-					<mesh filename="package://nao_meshes/meshes/V40/collision/${side}ShoulderPitch.ply"  scale="${scale} ${scale} ${scale}"/>
+				<origin xyz="0 0 0" rpy="-${PI_2} -0 0"/>
+				<geometry>
+					<mesh filename="package://nao_meshes/meshes/V40/visual/${side}ShoulderPitch.dae"  scale="${scale} ${scale} ${scale}"/>
+				</geometry>
+				<material name="LightGrey"/>
+			</visual>
+			<collision>
+				<origin xyz="0 0 0" rpy="0 -0 0"/>
+				<geometry>
+					<mesh filename="package://nao_meshes/meshes/V40/collision/${side}ShoulderPitch.dae"  scale="${scale} ${scale} ${scale}"/>
 				</geometry>
 				<material name="LightGrey"/>
@@ -136,14 +139,14 @@
 		<xacro:if value="${nao_meshes}">
 			<visual>
-				<origin xyz="0 0 0" rpy="0 -0 0"/>
-				<geometry>
-					<mesh filename="package://nao_meshes/meshes/V40/visual/${side}ShoulderRoll.obj"  scale="${scale} ${scale} ${scale}"/>
-				</geometry>
-				<material name="LightGrey"/>
-			</visual>
-			<collision>
-				<origin xyz="0 0 0" rpy="0 -0 0"/>
-				<geometry>
-					<mesh filename="package://nao_meshes/meshes/V40/collision/${side}ShoulderRoll.ply"  scale="${scale} ${scale} ${scale}"/>
+				<origin xyz="0 0 0" rpy="-${PI_2} -0 0"/>
+				<geometry>
+					<mesh filename="package://nao_meshes/meshes/V40/visual/${side}ShoulderRoll.dae"  scale="${scale} ${scale} ${scale}"/>
+				</geometry>
+				<material name="LightGrey"/>
+			</visual>
+			<collision>
+				<origin xyz="0 0 0" rpy="0 -0 0"/>
+				<geometry>
+					<mesh filename="package://nao_meshes/meshes/V40/collision/${side}ShoulderRoll.dae"  scale="${scale} ${scale} ${scale}"/>
 				</geometry>
 				<material name="LightGrey"/>
@@ -169,14 +172,14 @@
 		<xacro:if value="${nao_meshes}">
 			<visual>
-				<origin xyz="0 0 0" rpy="0 -0 0"/>
-				<geometry>
-					<mesh filename="package://nao_meshes/meshes/V40/visual/${side}ElbowRoll.obj"  scale="${scale} ${scale} ${scale}"/>
-				</geometry>
-				<material name="LightGrey"/>
-			</visual>
-			<collision>
-				<origin xyz="0 0 0" rpy="0 -0 0"/>
-				<geometry>
-					<mesh filename="package://nao_meshes/meshes/V40/collision/${side}ElbowRoll.ply"  scale="${scale} ${scale} ${scale}"/>
+				<origin xyz="0 0 0" rpy="-${PI_2} -0 0"/>
+				<geometry>
+					<mesh filename="package://nao_meshes/meshes/V40/visual/${side}ElbowRoll.dae"  scale="${scale} ${scale} ${scale}"/>
+				</geometry>
+				<material name="LightGrey"/>
+			</visual>
+			<collision>
+				<origin xyz="0 0 0" rpy="0 -0 0"/>
+				<geometry>
+					<mesh filename="package://nao_meshes/meshes/V40/collision/${side}ElbowRoll.dae"  scale="${scale} ${scale} ${scale}"/>
 				</geometry>
 				<material name="LightGrey"/>
@@ -202,14 +205,14 @@
 		<xacro:if value="${nao_meshes}">
 			<visual>
-				<origin xyz="0 0 0" rpy="0 -0 0"/>
-				<geometry>
-					<mesh filename="package://nao_meshes/meshes/V40/visual/WristYaw.obj"  scale="${scale} ${scale} ${scale}"/>
-				</geometry>
-				<material name="LightGrey"/>
-			</visual>
-			<collision>
-				<origin xyz="0 0 0" rpy="0 -0 0"/>
-				<geometry>
-					<mesh filename="package://nao_meshes/meshes/V40/collision/WristYaw.ply"  scale="${scale} ${scale} ${scale}"/>
+				<origin xyz="0 0 0" rpy="-${PI_2} -0 0"/>
+				<geometry>
+					<mesh filename="package://nao_meshes/meshes/V40/visual/WristYaw.dae"  scale="${scale} ${scale} ${scale}"/>
+				</geometry>
+				<material name="LightGrey"/>
+			</visual>
+			<collision>
+				<origin xyz="0 0 0" rpy="0 -0 0"/>
+				<geometry>
+					<mesh filename="package://nao_meshes/meshes/V40/collision/WristYaw.dae"  scale="${scale} ${scale} ${scale}"/>
 				</geometry>
 				<material name="LightGrey"/>
@@ -220,14 +223,14 @@
     	<xacro:if value="${nao_meshes}">
 			<visual>
-				<origin xyz="0 0 0" rpy="0 -0 0"/>
-				<geometry>
-					<mesh filename="package://nao_meshes/meshes/V40/visual/${side}HipYawPitch.obj"  scale="${scale} ${scale} ${scale}"/>
-				</geometry>
-				<material name="LightGrey"/>
-			</visual>
-			<collision>
-				<origin xyz="0 0 0" rpy="0 -0 0"/>
-				<geometry>
-					<mesh filename="package://nao_meshes/meshes/V40/collision/${side}HipYawPitch.ply"  scale="${scale} ${scale} ${scale}"/>
+				<origin xyz="0 0 0" rpy="-${PI_2} -0 0"/>
+				<geometry>
+					<mesh filename="package://nao_meshes/meshes/V40/visual/${side}HipYawPitch.dae"  scale="${scale} ${scale} ${scale}"/>
+				</geometry>
+				<material name="LightGrey"/>
+			</visual>
+			<collision>
+				<origin xyz="0 0 0" rpy="0 -0 0"/>
+				<geometry>
+					<mesh filename="package://nao_meshes/meshes/V40/collision/${side}HipYawPitch.dae"  scale="${scale} ${scale} ${scale}"/>
 				</geometry>
 				<material name="LightGrey"/>
@@ -238,14 +241,14 @@
     	<xacro:if value="${nao_meshes}">
 			<visual>
-				<origin xyz="0 0 0" rpy="0 -0 0"/>
-				<geometry>
-					<mesh filename="package://nao_meshes/meshes/V40/visual/${side}HipRoll.obj"  scale="${scale} ${scale} ${scale}"/>
-				</geometry>
-				<material name="LightGrey"/>
-			</visual>
-			<collision>
-				<origin xyz="0 0 0" rpy="0 -0 0"/>
-				<geometry>
-					<mesh filename="package://nao_meshes/meshes/V40/collision/${side}HipRoll.ply"  scale="${scale} ${scale} ${scale}"/>
+				<origin xyz="0 0 0" rpy="-${PI_2} -0 0"/>
+				<geometry>
+					<mesh filename="package://nao_meshes/meshes/V40/visual/${side}HipRoll.dae"  scale="${scale} ${scale} ${scale}"/>
+				</geometry>
+				<material name="LightGrey"/>
+			</visual>
+			<collision>
+				<origin xyz="0 0 0" rpy="0 -0 0"/>
+				<geometry>
+					<mesh filename="package://nao_meshes/meshes/V40/collision/${side}HipRoll.dae"  scale="${scale} ${scale} ${scale}"/>
 				</geometry>
 				<material name="LightGrey"/>
@@ -271,14 +274,14 @@
 		<xacro:if value="${nao_meshes}">
 			<visual>
-				<origin xyz="0 0 0" rpy="0 -0 0"/>
-				<geometry>
-					<mesh filename="package://nao_meshes/meshes/V40/visual/${side}HipPitch.obj"  scale="${scale} ${scale} ${scale}"/>
-				</geometry>
-				<material name="LightGrey"/>
-			</visual>
-			<collision>
-				<origin xyz="0 0 0" rpy="0 -0 0"/>
-				<geometry>
-					<mesh filename="package://nao_meshes/meshes/V40/collision/${side}HipPitch.ply"  scale="${scale} ${scale} ${scale}"/>
+				<origin xyz="0 0 0" rpy="-${PI_2} -0 0"/>
+				<geometry>
+					<mesh filename="package://nao_meshes/meshes/V40/visual/${side}HipPitch.dae"  scale="${scale} ${scale} ${scale}"/>
+				</geometry>
+				<material name="LightGrey"/>
+			</visual>
+			<collision>
+				<origin xyz="0 0 0" rpy="0 -0 0"/>
+				<geometry>
+					<mesh filename="package://nao_meshes/meshes/V40/collision/${side}HipPitch.dae"  scale="${scale} ${scale} ${scale}"/>
 				</geometry>
 				<material name="LightGrey"/>
@@ -304,14 +307,14 @@
 		<xacro:if value="${nao_meshes}">
 			<visual>
-				<origin xyz="0 0 0" rpy="0 -0 0"/>
-				<geometry>
-					<mesh filename="package://nao_meshes/meshes/V40/visual/${side}KneePitch.obj"  scale="${scale} ${scale} ${scale}"/>
-				</geometry>
-				<material name="LightGrey"/>
-			</visual>
-			<collision>
-				<origin xyz="0 0 0" rpy="0 -0 0"/>
-				<geometry>
-					<mesh filename="package://nao_meshes/meshes/V40/collision/${side}KneePitch.ply"  scale="${scale} ${scale} ${scale}"/>
+				<origin xyz="0 0 0" rpy="-${PI_2} -0 0"/>
+				<geometry>
+					<mesh filename="package://nao_meshes/meshes/V40/visual/${side}KneePitch.dae"  scale="${scale} ${scale} ${scale}"/>
+				</geometry>
+				<material name="LightGrey"/>
+			</visual>
+			<collision>
+				<origin xyz="0 0 0" rpy="0 -0 0"/>
+				<geometry>
+					<mesh filename="package://nao_meshes/meshes/V40/collision/${side}KneePitch.dae"  scale="${scale} ${scale} ${scale}"/>
 				</geometry>
 				<material name="LightGrey"/>
@@ -337,14 +340,14 @@
 		<xacro:if value="${nao_meshes}">
 			<visual>
-				<origin xyz="0 0 0" rpy="0 -0 0"/>
-				<geometry>
-					<mesh filename="package://nao_meshes/meshes/V40/visual/${side}AnklePitch.obj"  scale="${scale} ${scale} ${scale}"/>
-				</geometry>
-				<material name="LightGrey"/>
-			</visual>
-			<collision>
-				<origin xyz="0 0 0" rpy="0 -0 0"/>
-				<geometry>
-					<mesh filename="package://nao_meshes/meshes/V40/collision/${side}AnklePitch.ply"  scale="${scale} ${scale} ${scale}"/>
+				<origin xyz="0 0 0" rpy="-${PI_2} -0 0"/>
+				<geometry>
+					<mesh filename="package://nao_meshes/meshes/V40/visual/${side}AnklePitch.dae"  scale="${scale} ${scale} ${scale}"/>
+				</geometry>
+				<material name="LightGrey"/>
+			</visual>
+			<collision>
+				<origin xyz="0 0 0" rpy="0 -0 0"/>
+				<geometry>
+					<mesh filename="package://nao_meshes/meshes/V40/collision/${side}AnklePitch.dae"  scale="${scale} ${scale} ${scale}"/>
 				</geometry>
 				<material name="LightGrey"/>
@@ -370,14 +373,14 @@
 		<xacro:if value="${nao_meshes}">
 			<visual>
-				<origin xyz="0 0 0" rpy="0 -0 0"/>
-				<geometry>
-					<mesh filename="package://nao_meshes/meshes/V40/visual/${side}AnkleRoll.obj"  scale="${scale} ${scale} ${scale}"/>
-				</geometry>
-				<material name="LightGrey"/>
-			</visual>
-			<collision>
-				<origin xyz="0 0 0" rpy="0 -0 0"/>
-				<geometry>
-					<mesh filename="package://nao_meshes/meshes/V40/collision/${side}AnkleRoll.ply"  scale="${scale} ${scale} ${scale}"/>
+				<origin xyz="0 0 0" rpy="-${PI_2} -0 0"/>
+				<geometry>
+					<mesh filename="package://nao_meshes/meshes/V40/visual/${side}AnkleRoll.dae"  scale="${scale} ${scale} ${scale}"/>
+				</geometry>
+				<material name="LightGrey"/>
+			</visual>
+			<collision>
+				<origin xyz="0 0 0" rpy="0 -0 0"/>
+				<geometry>
+					<mesh filename="package://nao_meshes/meshes/V40/collision/${side}AnkleRoll.dae"  scale="${scale} ${scale} ${scale}"/>
 				</geometry>
 				<material name="LightGrey"/>
