Commit message: Added helmet_cameras_viz property to H25..

File: nao_dcm_common/nao_dcm_description/urdf/nao_dcm_H25.xacro (robot description, xacro)
@@ -8,4 +8,5 @@
 	<xacro:property name="nao_meshes" value="true" />
 	<xacro:property name="use_helmet" value="true" />
+	<xacro:property name="helmet_cameras_viz" value="false" />
 	<xacro:include filename="$(find nao_dcm_description)/urdf/nao_dcm_visuals_collisions.xacro" />
 	<xacro:include filename="$(find nao_dcm_description)/urdf/nao_dcm_gazebo.xacro" />
