Commit message: Changed URDF structure..

File: nao_dcm_common/nao_dcm_description/urdf/nao_dcm_H21.xacro (robot description, xacro)
@@ -5,7 +5,15 @@
 	<xacro:property name="PI_2" value="1.57079632679" />
 	<xacro:property name="scale" value="0.1" />
+	<xacro:property name="H25" value="false" />
 	<xacro:include filename="$(find nao_dcm_description)/urdf/nao_dcm_visuals_collisions.xacro" />
 	<xacro:include filename="$(find nao_dcm_description)/urdf/nao_dcm_gazebo.xacro" />
-	<xacro:include filename="$(find nao_dcm_description)/urdf/nao_dcm_H21_structure.xacro" />
 	<xacro:include filename="$(find nao_dcm_description)/urdf/nao_dcm_H21_control.xacro" />
+	<xacro:include filename="$(find nao_dcm_description)/urdf/modules/torso.xacro" />
+	<xacro:include filename="$(find nao_dcm_description)/urdf/modules/head.xacro" />
+	<xacro:include filename="$(find nao_dcm_description)/urdf/modules/arms.xacro" />
+	<xacro:include filename="$(find nao_dcm_description)/urdf/modules/hands.xacro" />
+	<xacro:include filename="$(find nao_dcm_description)/urdf/modules/legs.xacro" />
+	<xacro:include filename="$(find nao_dcm_description)/urdf/modules/imu.xacro" />
+	<xacro:include filename="$(find nao_dcm_description)/urdf/modules/sonars.xacro" />
+	<xacro:include filename="$(find nao_dcm_description)/urdf/modules/cameras.xacro" />
 </robot>

File: nao_dcm_common/nao_dcm_description/urdf/nao_dcm_H25.xacro (robot description, xacro)
@@ -5,7 +5,15 @@
 	<xacro:property name="PI_2" value="1.57079632679" />
 	<xacro:property name="scale" value="0.1" />
+	<xacro:property name="H25" value="true" />
 	<xacro:include filename="$(find nao_dcm_description)/urdf/nao_dcm_visuals_collisions.xacro" />
 	<xacro:include filename="$(find nao_dcm_description)/urdf/nao_dcm_gazebo.xacro" />
-	<xacro:include filename="$(find nao_dcm_description)/urdf/nao_dcm_H25_structure.xacro" />
 	<xacro:include filename="$(find nao_dcm_description)/urdf/nao_dcm_H25_control.xacro" />
+	<xacro:include filename="$(find nao_dcm_description)/urdf/modules/torso.xacro" />
+	<xacro:include filename="$(find nao_dcm_description)/urdf/modules/head.xacro" />
+	<xacro:include filename="$(find nao_dcm_description)/urdf/modules/arms.xacro" />
+	<xacro:include filename="$(find nao_dcm_description)/urdf/modules/hands.xacro" />
+	<xacro:include filename="$(find nao_dcm_description)/urdf/modules/legs.xacro" />
+	<xacro:include filename="$(find nao_dcm_description)/urdf/modules/imu.xacro" />
+	<xacro:include filename="$(find nao_dcm_description)/urdf/modules/sonars.xacro" />
+	<xacro:include filename="$(find nao_dcm_description)/urdf/modules/cameras.xacro" />
 </robot>

Commit message: Nao Helmet Added >3D Printed helmet for accessories on top of Nao's head added >Designed for adding cameras (in order to make stereo vision possible), but maybe can be used for other accessories too

File: nao_dcm_common/nao_dcm_description/urdf/nao_dcm_H21.xacro (robot description, xacro)
@@ -7,4 +7,6 @@
 	<xacro:property name="H25" value="false" />
 	<xacro:property name="nao_meshes" value="true" />
+	<xacro:property name="use_helmet" value="true" />
+	<xacro:property name="helmet_cameras_viz" value="false" />
 	<xacro:include filename="$(find nao_dcm_description)/urdf/nao_dcm_visuals_collisions.xacro" />
 	<xacro:include filename="$(find nao_dcm_description)/urdf/nao_dcm_gazebo.xacro" />
@@ -18,3 +20,7 @@
 	<xacro:include filename="$(find nao_dcm_description)/urdf/modules/sonars.xacro" />
 	<xacro:include filename="$(find nao_dcm_description)/urdf/modules/cameras.xacro" />
+	<xacro:if value="${use_helmet}">
+		<xacro:include filename="$(find nao_dcm_description)/urdf/modules/helmet.xacro" />
+		<xacro:include filename="$(find nao_dcm_description)/urdf/modules/helmet_cameras.xacro" />
+	</xacro:if>
 </robot>

File: nao_dcm_common/nao_dcm_description/urdf/nao_dcm_H25.xacro (robot description, xacro)
@@ -7,4 +7,5 @@
 	<xacro:property name="H25" value="true" />
 	<xacro:property name="nao_meshes" value="true" />
+	<xacro:property name="use_helmet" value="true" />
 	<xacro:include filename="$(find nao_dcm_description)/urdf/nao_dcm_visuals_collisions.xacro" />
 	<xacro:include filename="$(find nao_dcm_description)/urdf/nao_dcm_gazebo.xacro" />
@@ -18,3 +19,7 @@
 	<xacro:include filename="$(find nao_dcm_description)/urdf/modules/sonars.xacro" />
 	<xacro:include filename="$(find nao_dcm_description)/urdf/modules/cameras.xacro" />
+	<xacro:if value="${use_helmet}">
+		<xacro:include filename="$(find nao_dcm_description)/urdf/modules/helmet.xacro" />
+		<xacro:include filename="$(find nao_dcm_description)/urdf/modules/helmet_cameras.xacro" />
+	</xacro:if>
 </robot>

File: nao_dcm_common/nao_dcm_description/urdf/nao_dcm_visuals_collisions.xacro (robot description, xacro)
@@ -19,4 +19,20 @@
     <!-- END OF MATERIALS -->
     <!-- XACRO MACROS FOR VISUALS AND COLLISIONS -->
+    <xacro:macro name="visuals_collisions_helmet" params="">
+		<visual>
+			<origin xyz="0 0 0" rpy="0 -0 0"/>
+			<geometry>
+				<mesh filename="package://nao_dcm_description/meshes/helmet.dae"  scale="${scale} ${scale} ${scale}"/>
+			</geometry>
+			<material name="LightGrey"/>
+		</visual>
+		<collision>
+			<origin xyz="0 0 0" rpy="0 -0 0"/>
+			<geometry>
+				<mesh filename="package://nao_dcm_description/meshes/helmet.dae"  scale="${scale} ${scale} ${scale}"/>
+			</geometry>
+			<material name="LightGrey"/>
+		</collision>
+	</xacro:macro>
 	<xacro:macro name="visuals_collisions_torso" params="">
 		<xacro:unless value="${nao_meshes}">

Commit message: Added Ordoid 'Bag' in URDF..

File: nao_dcm_common/nao_dcm_description/urdf/nao_dcm_H21.xacro (robot description, xacro)
@@ -9,4 +9,5 @@
 	<xacro:property name="use_helmet" value="true" />
 	<xacro:property name="helmet_cameras_viz" value="false" />
+	<xacro:property name="use_odroid" value="true" />
 	<xacro:include filename="$(find nao_dcm_description)/urdf/nao_dcm_visuals_collisions.xacro" />
 	<xacro:include filename="$(find nao_dcm_description)/urdf/nao_dcm_gazebo.xacro" />
@@ -24,3 +25,6 @@
 		<xacro:include filename="$(find nao_dcm_description)/urdf/modules/helmet_cameras.xacro" />
 	</xacro:if>
+	<xacro:if value="${use_odroid}">
+		<xacro:include filename="$(find nao_dcm_description)/urdf/modules/odroid_bag.xacro" />
+	</xacro:if>
 </robot>

File: nao_dcm_common/nao_dcm_description/urdf/nao_dcm_H25.xacro (robot description, xacro)
@@ -9,4 +9,5 @@
 	<xacro:property name="use_helmet" value="true" />
 	<xacro:property name="helmet_cameras_viz" value="false" />
+	<xacro:property name="use_odroid" value="true" />
 	<xacro:include filename="$(find nao_dcm_description)/urdf/nao_dcm_visuals_collisions.xacro" />
 	<xacro:include filename="$(find nao_dcm_description)/urdf/nao_dcm_gazebo.xacro" />
@@ -24,3 +25,6 @@
 		<xacro:include filename="$(find nao_dcm_description)/urdf/modules/helmet_cameras.xacro" />
 	</xacro:if>
+	<xacro:if value="${use_odroid}">
+		<xacro:include filename="$(find nao_dcm_description)/urdf/modules/odroid_bag.xacro" />
+	</xacro:if>
 </robot>
