Commit message: Added odom publisher. Improved a little bit Gazebo integration

File: nao_dcm_common/nao_dcm_description/urdf/modules/helmet_cameras.xacro (robot description, xacro)
@@ -69,5 +69,5 @@
     <gazebo reference="LeftCamera">
         <sensor type="camera" name="LeftCamera">
-            <update_rate>10.0</update_rate>
+            <update_rate>30.0</update_rate>
             <camera name="left_camera">
                 <horizontal_fov>1.06290551</horizontal_fov>
@@ -89,5 +89,5 @@
             <plugin name="camera_controller" filename="libgazebo_ros_camera.so">
                 <alwaysOn>true</alwaysOn>
-                <updateRate>10.0</updateRate>
+                <updateRate>30.0</updateRate>
                 <cameraName>nao_dcm/CameraLeft</cameraName>
                 <imageTopicName>image_raw</imageTopicName>
@@ -105,5 +105,5 @@
     <gazebo reference="RightCamera">
         <sensor type="camera" name="RightCamera">
-            <update_rate>10.0</update_rate>
+            <update_rate>30.0</update_rate>
             <camera name="right_camera">
                 <horizontal_fov>1.06290551</horizontal_fov>
@@ -125,5 +125,5 @@
             <plugin name="camera_controller" filename="libgazebo_ros_camera.so">
                 <alwaysOn>true</alwaysOn>
-                <updateRate>10.0</updateRate>
+                <updateRate>30.0</updateRate>
                 <cameraName>nao_dcm/CameraRight</cameraName>
                 <imageTopicName>image_raw</imageTopicName>

File: nao_dcm_common/nao_dcm_description/urdf/nao_dcm_H21.xacro (robot description, xacro)
@@ -10,4 +10,11 @@
 	<xacro:property name="helmet_cameras_viz" value="false" />
 	<xacro:property name="use_odroid" value="true" />
+	<xacro:property name="use_hector_imu" value="false" />
+	<xacro:if value="${use_hector_imu}">
+		<xacro:property name="imu_plugin" value="libhector_gazebo_ros_imu.so" />
+	</xacro:if>
+	<xacro:unless value="${use_hector_imu}">
+		<xacro:property name="imu_plugin" value="libgazebo_ros_imu.so" />
+	</xacro:unless>
 	<xacro:include filename="$(find nao_dcm_description)/urdf/nao_dcm_visuals_collisions.xacro" />
 	<xacro:include filename="$(find nao_dcm_description)/urdf/nao_dcm_gazebo.xacro" />

File: nao_dcm_common/nao_dcm_description/urdf/nao_dcm_H25.xacro (robot description, xacro)
@@ -10,4 +10,11 @@
 	<xacro:property name="helmet_cameras_viz" value="false" />
 	<xacro:property name="use_odroid" value="true" />
+	<xacro:property name="use_hector_imu" value="false" />
+	<xacro:if value="${use_hector_imu}">
+		<xacro:property name="imu_plugin" value="libhector_gazebo_ros_imu.so" />
+	</xacro:if>
+	<xacro:unless value="${use_hector_imu}">
+		<xacro:property name="imu_plugin" value="libgazebo_ros_imu.so" />
+	</xacro:unless>
 	<xacro:include filename="$(find nao_dcm_description)/urdf/nao_dcm_visuals_collisions.xacro" />
 	<xacro:include filename="$(find nao_dcm_description)/urdf/nao_dcm_gazebo.xacro" />

File: nao_dcm_common/nao_dcm_description/urdf/nao_dcm_gazebo.xacro (robot description, xacro)
@@ -7,9 +7,13 @@
             <robotSimType>gazebo_ros_control/DefaultRobotHWSim</robotSimType>
         </plugin>
-        <plugin name="gazebo_ros_imu_controller" filename="libgazebo_ros_imu.so">
+        <plugin name="gazebo_ros_imu_controller" filename="${imu_plugin}">
             <robotNamespace>/nao_dcm</robotNamespace>
             <topicName>imu_data</topicName>
             <bodyName>imu</bodyName>
+            <frameId>imu</frameId>
             <gaussianNoise>2.89e-08</gaussianNoise>
+            <accelGaussianNoise>2.89e-08 2.89e-08 2.89e-08</accelGaussianNoise>
+            <rateGaussianNoise>2.89e-08 2.89e-08 2.89e-08</rateGaussianNoise>
+            <headingGaussianNoise>2.89e-08 2.89e-08 2.89e-08</headingGaussianNoise>
             <xyzOffsets>0 0 0</xyzOffsets>
             <rpyOffsets>0 0 0</rpyOffsets>
