Commit message: Added fingers to URDF and Gazebo..Integration with MimicJointPlugin for adding mimic joints to Gazebo

File: nao_dcm_common/nao_dcm_description/urdf/modules/hands.xacro (robot description, xacro)
@@ -1,4 +1,101 @@
 <?xml version="1.0"?>
 <robot xmlns:xacro="http://www.ros.org/wiki/xacro">
+	<!-- Fingers -->
+	<xacro:macro name="Finger" params="side num side_small reflect">
+		<joint name="${side}Finger${num}" type="revolute">
+	    	<parent link="${side_small}_wrist"/>
+	    	<child link="${side}Finger${num}1"/>
+	    	<origin xyz="0.06907 ${reflect*0.01157} -0.00304" rpy="0 0 0"/>
+	    	<axis xyz="0 1 0"/>
+	    	<mimic joint="${side}Hand" multiplier="-${PI/4}" offset="${PI/4}"/>
+	    	<!-- Dummy values for mimic joint -->
+	    	<limit effort="10.0" lower="0.0" upper="${PI/4}" velocity="3.0"/>
+	    </joint>
+	    <link name="${side}Finger${num}1">
+	    	<xacro:visuals_collisions_phalax reflect="-1" side="${side}"/>
+	    	<inertial> <!-- dummy values for gazebo -->
+	            <mass value="0.2e-5" />
+	            <origin xyz="0 0 0"/>
+	            <inertia ixx="1e-9" ixy="0" ixz="0" iyy="1e-9" iyz="0" izz="1e-9" />
+	        </inertial>
+	    </link>
+	    <joint name="${side}Finger${num}_1" type="revolute">
+	    	<parent link="${side}Finger${num}1"/>
+	    	<child link="${side}Finger${num}2"/>
+	    	<origin xyz="0.01436 0 0" rpy="0 0 0"/>
+	    	<axis xyz="0 1 0"/>
+	    	<mimic joint="${side}Hand" multiplier="-${PI/4}" offset="${PI/4}"/>
+	    	<!-- Dummy values for mimic joint -->
+	    	<limit effort="10.0" lower="0.0" upper="${PI/4}" velocity="3.0"/>
+	    </joint>
+	    <link name="${side}Finger${num}2">
+	    	<xacro:visuals_collisions_phalax reflect="-1" side="${side}"/>
+	    	<inertial> <!-- dummy values for gazebo -->
+	            <mass value="0.2e-5" />
+	            <origin xyz="0 0 0"/>
+	            <inertia ixx="1e-9" ixy="0" ixz="0" iyy="1e-9" iyz="0" izz="1e-9" />
+	        </inertial>
+	    </link>
+	    <joint name="${side}Finger${num}_2" type="revolute">
+	    	<parent link="${side}Finger${num}2"/>
+	    	<child link="${side}Finger${num}3"/>
+	    	<origin xyz="0.01436 0 0" rpy="0 0 0"/>
+	    	<axis xyz="0 1 0"/>
+	    	<mimic joint="${side}Hand" multiplier="-${PI/4}" offset="${PI/4}"/>
+	    	<!-- Dummy values for mimic joint -->
+	    	<limit effort="10.0" lower="0.0" upper="${PI/4}" velocity="3.0"/>
+	    </joint>
+	    <link name="${side}Finger${num}3">
+	    	<xacro:visuals_collisions_phalax_end reflect="-1" side="${side}"/>
+	    	<inertial> <!-- dummy values for gazebo -->
+	            <mass value="0.2e-5" />
+	            <origin xyz="0 0 0"/>
+	            <inertia ixx="1e-9" ixy="0" ixz="0" iyy="1e-9" iyz="0" izz="1e-9" />
+	        </inertial>
+	    </link>
+	</xacro:macro>
+	<xacro:Finger side="L" side_small="l" num="1" reflect="1"/>
+	<xacro:Finger side="L" side_small="l" num="2" reflect="-1"/>
+	<xacro:Finger side="R" side_small="r" num="1" reflect="1"/>
+	<xacro:Finger side="R" side_small="r" num="2" reflect="-1"/>
+	<!-- Thumbs -->
+	<xacro:macro name="Thumb" params="side side_small">
+		<joint name="${side}Thumb1_joint" type="revolute">
+	    	<parent link="${side_small}_wrist"/>
+	    	<child link="${side}Thumb1"/>
+	    	<origin xyz="0.04895 0 -0.02638" rpy="${PI} ${PI/4} 0"/>
+	    	<axis xyz="0 1 0"/>
+	    	<mimic joint="${side}Hand" multiplier="-${PI/4}" offset="${PI/4}"/>
+	    	<!-- Dummy values for mimic joint -->
+	    	<limit effort="10.0" lower="0.0" upper="${PI/4}" velocity="3.0"/>
+	    </joint>
+	    <link name="${side}Thumb1">
+	    	<xacro:visuals_collisions_phalax reflect="-1" side="${side}"/>
+	    	<inertial> <!-- dummy values for gazebo -->
+	            <mass value="0.2e-5" />
+	            <origin xyz="0 0 0"/>
+	            <inertia ixx="1e-9" ixy="0" ixz="0" iyy="1e-9" iyz="0" izz="1e-9" />
+	        </inertial>
+	    </link>
+	    <joint name="${side}Thumb1_2" type="revolute">
+	    	<parent link="${side}Thumb1"/>
+	    	<child link="${side}Thumb2"/>
+	    	<origin xyz="0.01436 0 0" rpy="0 0 0"/>
+	    	<axis xyz="0 1 0"/>
+	    	<mimic joint="${side}Hand" multiplier="-${PI/4}" offset="${PI/4}"/>
+	    	<!-- Dummy values for mimic joint -->
+	    	<limit effort="10.0" lower="0.0" upper="${PI/4}" velocity="3.0"/>
+	    </joint>
+	    <link name="${side}Thumb2">
+	    	<xacro:visuals_collisions_phalax_end reflect="-1" side="${side}"/>
+	    	<inertial> <!-- dummy values for gazebo -->
+	            <mass value="0.2e-5" />
+	            <origin xyz="0 0 0"/>
+	            <inertia ixx="1e-9" ixy="0" ixz="0" iyy="1e-9" iyz="0" izz="1e-9" />
+	        </inertial>
+	    </link>
+	</xacro:macro>
+	<xacro:Thumb side="L" side_small="l"/>
+	<xacro:Thumb side="R" side_small="r"/>
 	<!-- H25 Hands -->
 	<xacro:if value="${H25}">
@@ -92,4 +189,32 @@
 	        </inertial>
 	    </link>
+	    <!-- DUMMY REVOLUTE JOINT FOR NON MOTORED HAND -->
+	    <joint name="LHand" type="revolute">
+	        <parent link="l_wrist"/>
+	        <child link="l_gripper"/>
+	        <origin rpy="0 0 0" xyz="0.05775 0 0"/>
+	        <limit effort="10.0" lower="0.0" upper="0.0" velocity="3.0"/>
+	    </joint>
+	    <link name="l_gripper">
+	        <inertial> <!-- dummy values for gazebo -->
+	            <mass value="0.2e-5" />
+	            <origin xyz="0 0 0"/>
+	            <inertia ixx="1e-9" ixy="0" ixz="0" iyy="1e-9" iyz="0" izz="1e-9" />
+	        </inertial>
+	    </link>
+	    <!-- DUMMY REVOLUTE JOINT FOR NON MOTORED HAND -->
+	    <joint name="RHand" type="revolute">
+	        <parent link="r_wrist"/>
+	        <child link="r_gripper"/>
+	        <origin rpy="0 0 0" xyz="0.05775 0 0"/>
+	        <limit effort="10.0" lower="0.0" upper="0.0" velocity="3.0"/>
+	    </joint>
+	    <link name="r_gripper">
+	        <inertial> <!-- dummy values for gazebo -->
+	            <mass value="0.2e-5" />
+	            <origin xyz="0 0 0"/>
+	            <inertia ixx="1e-9" ixy="0" ixz="0" iyy="1e-9" iyz="0" izz="1e-9" />
+	        </inertial>
+	    </link>
 	</xacro:unless>
 </robot>

File: nao_dcm_common/nao_dcm_description/urdf/nao_dcm_H21.xacro (robot description, xacro)
@@ -2,36 +2,6 @@
 <robot name="nao_robot_v4_H21" xmlns:xacro="http://www.ros.org/wiki/xacro">
 	<!-- XACRO PROPERTIES -->
-	<xacro:property name="PI" value="3.14159265359" />
-	<xacro:property name="PI_2" value="1.57079632679" />
-	<xacro:property name="scale" value="0.001" />
 	<xacro:property name="H25" value="false" />
-	<xacro:property name="nao_meshes" value="true" />
-	<xacro:property name="use_helmet" value="true" />
-	<xacro:property name="helmet_cameras_viz" value="false" />
-	<xacro:property name="use_odroid" value="true" />
-	<xacro:property name="use_hector_imu" value="false" />
-	<xacro:if value="${use_hector_imu}">
-		<xacro:property name="imu_plugin" value="libhector_gazebo_ros_imu.so" />
-	</xacro:if>
-	<xacro:unless value="${use_hector_imu}">
-		<xacro:property name="imu_plugin" value="libgazebo_ros_imu.so" />
-	</xacro:unless>
-	<xacro:include filename="$(find nao_dcm_description)/urdf/nao_dcm_visuals_collisions.xacro" />
-	<xacro:include filename="$(find nao_dcm_description)/urdf/nao_dcm_gazebo.xacro" />
 	<xacro:include filename="$(find nao_dcm_description)/urdf/nao_dcm_H21_control.xacro" />
-	<xacro:include filename="$(find nao_dcm_description)/urdf/modules/torso.xacro" />
-	<xacro:include filename="$(find nao_dcm_description)/urdf/modules/head.xacro" />
-	<xacro:include filename="$(find nao_dcm_description)/urdf/modules/arms.xacro" />
-	<xacro:include filename="$(find nao_dcm_description)/urdf/modules/hands.xacro" />
-	<xacro:include filename="$(find nao_dcm_description)/urdf/modules/legs.xacro" />
-	<xacro:include filename="$(find nao_dcm_description)/urdf/modules/imu.xacro" />
-	<xacro:include filename="$(find nao_dcm_description)/urdf/modules/sonars.xacro" />
-	<xacro:include filename="$(find nao_dcm_description)/urdf/modules/cameras.xacro" />
-	<xacro:if value="${use_helmet}">
-		<xacro:include filename="$(find nao_dcm_description)/urdf/modules/helmet.xacro" />
-		<xacro:include filename="$(find nao_dcm_description)/urdf/modules/helmet_cameras.xacro" />
-	</xacro:if>
-	<xacro:if value="${use_odroid}">
-		<xacro:include filename="$(find nao_dcm_description)/urdf/modules/odroid_bag.xacro" />
-	</xacro:if>
+	<xacro:include filename="$(find nao_dcm_description)/urdf/modules/robot.xacro" />
 </robot>

File: nao_dcm_common/nao_dcm_description/urdf/nao_dcm_H25.xacro (robot description, xacro)
@@ -2,36 +2,6 @@
 <robot name="nao_robot_v4_H25" xmlns:xacro="http://www.ros.org/wiki/xacro">
 	<!-- XACRO PROPERTIES -->
-	<xacro:property name="PI" value="3.14159265359" />
-	<xacro:property name="PI_2" value="1.57079632679" />
-	<xacro:property name="scale" value="0.001" />
 	<xacro:property name="H25" value="true" />
-	<xacro:property name="nao_meshes" value="true" />
-	<xacro:property name="use_helmet" value="true" />
-	<xacro:property name="helmet_cameras_viz" value="false" />
-	<xacro:property name="use_odroid" value="true" />
-	<xacro:property name="use_hector_imu" value="false" />
-	<xacro:if value="${use_hector_imu}">
-		<xacro:property name="imu_plugin" value="libhector_gazebo_ros_imu.so" />
-	</xacro:if>
-	<xacro:unless value="${use_hector_imu}">
-		<xacro:property name="imu_plugin" value="libgazebo_ros_imu.so" />
-	</xacro:unless>
-	<xacro:include filename="$(find nao_dcm_description)/urdf/nao_dcm_visuals_collisions.xacro" />
-	<xacro:include filename="$(find nao_dcm_description)/urdf/nao_dcm_gazebo.xacro" />
 	<xacro:include filename="$(find nao_dcm_description)/urdf/nao_dcm_H25_control.xacro" />
-	<xacro:include filename="$(find nao_dcm_description)/urdf/modules/torso.xacro" />
-	<xacro:include filename="$(find nao_dcm_description)/urdf/modules/head.xacro" />
-	<xacro:include filename="$(find nao_dcm_description)/urdf/modules/arms.xacro" />
-	<xacro:include filename="$(find nao_dcm_description)/urdf/modules/hands.xacro" />
-	<xacro:include filename="$(find nao_dcm_description)/urdf/modules/legs.xacro" />
-	<xacro:include filename="$(find nao_dcm_description)/urdf/modules/imu.xacro" />
-	<xacro:include filename="$(find nao_dcm_description)/urdf/modules/sonars.xacro" />
-	<xacro:include filename="$(find nao_dcm_description)/urdf/modules/cameras.xacro" />
-	<xacro:if value="${use_helmet}">
-		<xacro:include filename="$(find nao_dcm_description)/urdf/modules/helmet.xacro" />
-		<xacro:include filename="$(find nao_dcm_description)/urdf/modules/helmet_cameras.xacro" />
-	</xacro:if>
-	<xacro:if value="${use_odroid}">
-		<xacro:include filename="$(find nao_dcm_description)/urdf/modules/odroid_bag.xacro" />
-	</xacro:if>
+	<xacro:include filename="$(find nao_dcm_description)/urdf/modules/robot.xacro" />
 </robot>

File: nao_dcm_common/nao_dcm_description/urdf/nao_dcm_gazebo.xacro (robot description, xacro)
@@ -1,4 +1,41 @@
 <?xml version="1.0"?>
 <robot xmlns:xacro="http://www.ros.org/wiki/xacro">
+    <!-- MACROS FOR MIMIC JOINTS -->
+    <!-- Fingers -->
+    <xacro:macro name="FingerMimics" params="side num">
+        <plugin name="mimic_${side}Finger${num}" filename="libgazebo_mimic_joint_plugin.so">
+            <joint>${side}Hand</joint>
+            <mimicJoint>${side}Finger${num}</mimicJoint>
+            <multiplier>-${PI/4}</multiplier>
+            <offset>${PI/4}</offset>
+        </plugin>
+        <plugin name="mimic_${side}Finger${num}_1" filename="libgazebo_mimic_joint_plugin.so">
+            <joint>${side}Hand</joint>
+            <mimicJoint>${side}Finger${num}_1</mimicJoint>
+            <multiplier>-${PI/4}</multiplier>
+            <offset>${PI/4}</offset>
+        </plugin>
+        <plugin name="mimic_${side}Finger${num}_2" filename="libgazebo_mimic_joint_plugin.so">
+            <joint>${side}Hand</joint>
+            <mimicJoint>${side}Finger${num}_2</mimicJoint>
+            <multiplier>-${PI/4}</multiplier>
+            <offset>${PI/4}</offset>
+        </plugin>
+    </xacro:macro>
+    <!-- Thumbs -->
+    <xacro:macro name="ThumbMimics" params="side">
+        <plugin name="${side}Thumb1_joint" filename="libgazebo_mimic_joint_plugin.so">
+            <joint>${side}Hand</joint>
+            <mimicJoint>${side}Thumb1_joint</mimicJoint>
+            <multiplier>-${PI/4}</multiplier>
+            <offset>${PI/4}</offset>
+        </plugin>
+        <plugin name="${side}Thumb1_2" filename="libgazebo_mimic_joint_plugin.so">
+            <joint>${side}Hand</joint>
+            <mimicJoint>${side}Thumb1_2</mimicJoint>
+            <multiplier>-${PI/4}</multiplier>
+            <offset>${PI/4}</offset>
+        </plugin>
+    </xacro:macro>
     <!-- GAZEBO ROS CONTROL AND IMU PLUGIN -->
     <gazebo>
@@ -21,4 +58,17 @@
             <alwaysOn>true</alwaysOn>
         </plugin>
+        <!-- Mimic joints through plugin develop by costashatz based on implementation by Goncalo Cabrita -->
+        <plugin name="mimic_hipyawpitch" filename="libgazebo_mimic_joint_plugin.so">
+            <joint>LHipYawPitch</joint>
+            <mimicJoint>RHipYawPitch</mimicJoint>
+            <multiplier>1.0</multiplier>
+            <offset>0.0</offset>
+        </plugin>
+        <xacro:FingerMimics side="L" num="1"/>
+        <xacro:FingerMimics side="L" num="2"/>
+        <xacro:FingerMimics side="R" num="1"/>
+        <xacro:FingerMimics side="R" num="2"/>
+        <xacro:ThumbMimics side="L"/>
+        <xacro:ThumbMimics side="R"/>
     </gazebo>
     <!-- END OF GAZEBO ROS CONTROL PLUGIN -->
@@ -85,4 +135,60 @@
         <turnGravityOff>false</turnGravityOff>
     </gazebo>
+    <gazebo reference="LFinger11">
+        <material>Gazebo/Yellow</material>
+        <mu1>0.5</mu1>
+        <mu2>0.5</mu2>
+        <selfCollide>false</selfCollide>
+        <turnGravityOff>false</turnGravityOff>
+    </gazebo>
+    <gazebo reference="LFinger12">
+        <material>Gazebo/Yellow</material>
+        <mu1>0.5</mu1>
+        <mu2>0.5</mu2>
+        <selfCollide>false</selfCollide>
+        <turnGravityOff>false</turnGravityOff>
+    </gazebo>
+    <gazebo reference="LFinger13">
+        <material>Gazebo/Yellow</material>
+        <mu1>0.5</mu1>
+        <mu2>0.5</mu2>
+        <selfCollide>false</selfCollide>
+        <turnGravityOff>false</turnGravityOff>
+    </gazebo>
+    <gazebo reference="LFinger21">
+        <material>Gazebo/Yellow</material>
+        <mu1>0.5</mu1>
+        <mu2>0.5</mu2>
+        <selfCollide>false</selfCollide>
+        <turnGravityOff>false</turnGravityOff>
+    </gazebo>
+    <gazebo reference="LFinger22">
+        <material>Gazebo/Yellow</material>
+        <mu1>0.5</mu1>
+        <mu2>0.5</mu2>
+        <selfCollide>false</selfCollide>
+        <turnGravityOff>false</turnGravityOff>
+    </gazebo>
+    <gazebo reference="LFinger23">
+        <material>Gazebo/Yellow</material>
+        <mu1>0.5</mu1>
+        <mu2>0.5</mu2>
+        <selfCollide>false</selfCollide>
+        <turnGravityOff>false</turnGravityOff>
+    </gazebo>
+    <gazebo reference="LThumb1">
+        <material>Gazebo/Yellow</material>
+        <mu1>0.5</mu1>
+        <mu2>0.5</mu2>
+        <selfCollide>false</selfCollide>
+        <turnGravityOff>false</turnGravityOff>
+    </gazebo>
+    <gazebo reference="LThumb2">
+        <material>Gazebo/Yellow</material>
+        <mu1>0.5</mu1>
+        <mu2>0.5</mu2>
+        <selfCollide>false</selfCollide>
+        <turnGravityOff>false</turnGravityOff>
+    </gazebo>
     <gazebo reference="l_gripper">
         <material>Gazebo/Yellow</material>
@@ -112,4 +218,60 @@
     </gazebo>
     <gazebo reference="r_wrist">
+        <material>Gazebo/Yellow</material>
+        <mu1>0.5</mu1>
+        <mu2>0.5</mu2>
+        <selfCollide>false</selfCollide>
+        <turnGravityOff>false</turnGravityOff>
+    </gazebo>
+    <gazebo reference="RFinger11">
+        <material>Gazebo/Yellow</material>
+        <mu1>0.5</mu1>
+        <mu2>0.5</mu2>
+        <selfCollide>false</selfCollide>
+        <turnGravityOff>false</turnGravityOff>
+    </gazebo>
+    <gazebo reference="RFinger12">
+        <material>Gazebo/Yellow</material>
+        <mu1>0.5</mu1>
+        <mu2>0.5</mu2>
+        <selfCollide>false</selfCollide>
+        <turnGravityOff>false</turnGravityOff>
+    </gazebo>
+    <gazebo reference="RFinger13">
+        <material>Gazebo/Yellow</material>
+        <mu1>0.5</mu1>
+        <mu2>0.5</mu2>
+        <selfCollide>false</selfCollide>
+        <turnGravityOff>false</turnGravityOff>
+    </gazebo>
+    <gazebo reference="RFinger21">
+        <material>Gazebo/Yellow</material>
+        <mu1>0.5</mu1>
+        <mu2>0.5</mu2>
+        <selfCollide>false</selfCollide>
+        <turnGravityOff>false</turnGravityOff>
+    </gazebo>
+    <gazebo reference="RFinger22">
+        <material>Gazebo/Yellow</material>
+        <mu1>0.5</mu1>
+        <mu2>0.5</mu2>
+        <selfCollide>false</selfCollide>
+        <turnGravityOff>false</turnGravityOff>
+    </gazebo>
+    <gazebo reference="RFinger23">
+        <material>Gazebo/Yellow</material>
+        <mu1>0.5</mu1>
+        <mu2>0.5</mu2>
+        <selfCollide>false</selfCollide>
+        <turnGravityOff>false</turnGravityOff>
+    </gazebo>
+    <gazebo reference="RThumb1">
+        <material>Gazebo/Yellow</material>
+        <mu1>0.5</mu1>
+        <mu2>0.5</mu2>
+        <selfCollide>false</selfCollide>
+        <turnGravityOff>false</turnGravityOff>
+    </gazebo>
+    <gazebo reference="RThumb2">
         <material>Gazebo/Yellow</material>
         <mu1>0.5</mu1>

File: nao_dcm_common/nao_dcm_description/urdf/nao_dcm_visuals_collisions.xacro (robot description, xacro)
@@ -236,4 +236,70 @@
 		</xacro:if>
     </xacro:macro>
+    <xacro:macro name="visuals_collisions_phalax" params="side reflect">
+    	<xacro:unless value="${nao_meshes}">
+			<visual>
+				<origin xyz="0.000718 0 0" rpy="${PI_2} 0 ${PI_2}"/>
+	            <geometry>
+	                <box size="0.01 0.01 0.01436"/>
+	            </geometry>
+				<material name="Yellow"/>
+			</visual>
+			<collision>
+				<origin xyz="0.000718 0 0" rpy="${PI_2} 0 ${PI_2}"/>
+	            <geometry>
+	                <box size="0.01 0.01 0.01436"/>
+	            </geometry>
+			</collision>
+		</xacro:unless>
+		<xacro:if value="${nao_meshes}">
+			<visual>
+				<origin xyz="0 0 0" rpy="-${PI_2} -0 0"/>
+				<geometry>
+					<mesh filename="package://nao_meshes/meshes/V40/visual/Phalax.dae"  scale="${scale} ${scale} ${scale}"/>
+				</geometry>
+				<material name="LightGrey"/>
+			</visual>
+			<collision>
+				<origin xyz="0 0 0" rpy="0 -0 0"/>
+				<geometry>
+					<mesh filename="package://nao_meshes/meshes/V40/collision/Phalax.dae"  scale="${scale} ${scale} ${scale}"/>
+				</geometry>
+				<material name="LightGrey"/>
+			</collision>
+		</xacro:if>
+    </xacro:macro>
+    <xacro:macro name="visuals_collisions_phalax_end" params="side reflect">
+    	<xacro:unless value="${nao_meshes}">
+			<visual>
+				<origin xyz="0.000718 0 0" rpy="${PI_2} 0 ${PI_2}"/>
+	            <geometry>
+	                <box size="0.01 0.01 0.01436"/>
+	            </geometry>
+				<material name="Yellow"/>
+			</visual>
+			<collision>
+				<origin xyz="0.000718 0 0" rpy="${PI_2} 0 ${PI_2}"/>
+	            <geometry>
+	                <box size="0.01 0.01 0.01436"/>
+	            </geometry>
+			</collision>
+		</xacro:unless>
+		<xacro:if value="${nao_meshes}">
+			<visual>
+				<origin xyz="0 0 0" rpy="-${PI_2} -0 0"/>
+				<geometry>
+					<mesh filename="package://nao_meshes/meshes/V40/visual/PhalaxEnd.dae"  scale="${scale} ${scale} ${scale}"/>
+				</geometry>
+				<material name="LightGrey"/>
+			</visual>
+			<collision>
+				<origin xyz="0 0 0" rpy="0 -0 0"/>
+				<geometry>
+					<mesh filename="package://nao_meshes/meshes/V40/collision/PhalaxEnd.dae"  scale="${scale} ${scale} ${scale}"/>
+				</geometry>
+				<material name="LightGrey"/>
+			</collision>
+		</xacro:if>
+    </xacro:macro>
     <xacro:macro name="visuals_collisions_hip_yaw_pitch" params="side reflect">
     	<xacro:if value="${nao_meshes}">
