Commit message: URDF /xacro more modular. Small gazebo improvements. Updates in README

File: nao_dcm_common/nao_dcm_description/urdf/modules/arms.xacro (robot description, xacro)
@@ -44,5 +44,5 @@
             <parent link="torso"/>
             <child link="${side}Shoulder"/>
-            <limit effort="${150.27*14.3/1000.0}" lower="-2.0857" upper="2.0857" velocity="3.0"/>
+            <limit effort="${effort_type3*speed_red_type3A}" lower="-2.0857" upper="2.0857" velocity="3.0"/>
             <origin rpy="0 0 0" xyz="0 ${reflect*0.098} 0.1"/>
             <axis xyz="0 1 0"/>
@@ -60,5 +60,5 @@
             <parent link="${side}ShoulderDummy"/>
             <child link="${side}Elbow"/>
-            <limit effort="${150.27*14.3/1000.0}" lower="-2.0857" upper="2.0857" velocity="3.0"/>
+            <limit effort="${effort_type3*speed_red_type3A}" lower="-2.0857" upper="2.0857" velocity="3.0"/>
             <origin rpy="0 0 0" xyz="0.105 ${reflect*0.015} 0"/>
             <axis xyz="1 0 0"/>
@@ -79,5 +79,5 @@
         <parent link="LShoulder"/>
         <child link="LShoulderDummy"/>
-        <limit effort="${173.22*14.3/1000.0}" lower="-0.3142" upper="1.3265" velocity="3.0"/>
+        <limit effort="${effort_type3*speed_red_type3B}" lower="-0.3142" upper="1.3265" velocity="3.0"/>
         <origin rpy="0 0 0" xyz="0 0 0"/>
         <axis xyz="0 0 1"/>
@@ -86,5 +86,5 @@
         <parent link="RShoulder"/>
         <child link="RShoulderDummy"/>
-        <limit effort="${173.22*14.3/1000.0}" lower="-1.3265" upper="0.3142" velocity="3.0"/>
+        <limit effort="${effort_type3*speed_red_type3B}" lower="-1.3265" upper="0.3142" velocity="3.0"/>
         <origin rpy="0 0 0" xyz="0 0 0"/>
         <axis xyz="0 0 1"/>
@@ -93,5 +93,5 @@
         <parent link="LElbow"/>
         <child link="LElbowDummy"/>
-        <limit effort="${173.22*14.3/1000.0}" lower="-1.5446" upper="-0.0349" velocity="3.0"/>
+        <limit effort="${effort_type3*speed_red_type3B}" lower="-1.5446" upper="-0.0349" velocity="3.0"/>
         <origin rpy="0 0 0" xyz="0 0 0"/>
         <axis xyz="0 0 1"/>
@@ -100,5 +100,5 @@
         <parent link="RElbow"/>
         <child link="RElbowDummy"/>
-        <limit effort="${173.22*14.3/1000.0}" lower="0.0349" upper="1.5446" velocity="3.0"/>
+        <limit effort="${effort_type3*speed_red_type3B}" lower="0.0349" upper="1.5446" velocity="3.0"/>
         <origin rpy="0 0 0" xyz="0 0 0"/>
         <axis xyz="0 0 1"/>

File: nao_dcm_common/nao_dcm_description/urdf/modules/hands.xacro (robot description, xacro)
@@ -104,5 +104,5 @@
 	        <child link="l_wrist"/>
 	        <origin rpy="0 0 0" xyz="0.05595 0 0"/>
-	        <limit effort="${50.61*9.4/1000.0}" lower="-1.8238" upper="1.8238" velocity="3.0"/>
+	        <limit effort="${effort_type2*speed_red_type2A}" lower="-1.8238" upper="1.8238" velocity="3.0"/>
 	    </joint>
 	    <link name="l_wrist">
@@ -120,5 +120,5 @@
 	        <child link="l_gripper"/>
 	        <origin rpy="0 0 0" xyz="0.05775 0 0"/>
-	        <limit effort="${36.24*9.4/1000.0}" lower="0.0" upper="1.0" velocity="3.0"/>
+	        <limit effort="${effort_type2*speed_red_type2B}" lower="0.0" upper="1.0" velocity="3.0"/>
 	    </joint>
 	    <link name="l_gripper">
@@ -133,5 +133,5 @@
 	        <child link="r_wrist"/>
 	        <origin rpy="0 0 0" xyz="0.05595 0 0"/>
-	        <limit effort="${50.61*9.4/1000.0}" lower="-1.8238" upper="1.8238" velocity="3.0"/>
+	        <limit effort="${effort_type2*speed_red_type2A}" lower="-1.8238" upper="1.8238" velocity="3.0"/>
 	    </joint>
 	    <link name="r_wrist">
@@ -149,5 +149,5 @@
 	        <child link="r_gripper"/>
 	        <origin rpy="0 0 0" xyz="0.05775 0 0"/>
-	        <limit effort="${36.24*9.4/1000.0}" lower="0.0" upper="1.0" velocity="3.0"/>
+	        <limit effort="${effort_type2*speed_red_type2B}" lower="0.0" upper="1.0" velocity="3.0"/>
 	    </joint>
 	    <link name="r_gripper">

File: nao_dcm_common/nao_dcm_description/urdf/modules/head.xacro (robot description, xacro)
@@ -5,5 +5,5 @@
         <parent link="torso"/>
         <child link="neck"/>
-        <limit effort="${150.27*14.3/1000.0}" lower="-2.0857" upper="2.0857" velocity="3.0"/>
+        <limit effort="${effort_type3*speed_red_type3A}" lower="-2.0857" upper="2.0857" velocity="3.0"/>
         <origin rpy="0 0 0" xyz="0 0 0.1265"/>
         <axis xyz="0 0 1"/>
@@ -22,5 +22,5 @@
         <parent link="neck"/>
         <child link="gaze"/>
-        <limit effort="${173.22*14.3/1000.0}" lower="-0.6720" upper="0.5149" velocity="3.0"/>
+        <limit effort="${effort_type3*speed_red_type3B}" lower="-0.6720" upper="0.5149" velocity="3.0"/>
         <origin rpy="0 0 0" xyz="0 0 0"/>
         <axis xyz="0 1 0"/>

File: nao_dcm_common/nao_dcm_description/urdf/modules/legs.xacro (robot description, xacro)
@@ -5,5 +5,5 @@
         <parent link="base_link"/>
         <child link="LHipYaw"/>
-        <limit effort="${201.3*68/1000.0}" lower="-1.145303" upper="0.740810" velocity="3.0"/>
+        <limit effort="${effort_type1*speed_red_type1A}" lower="-1.145303" upper="0.740810" velocity="3.0"/>
         <origin rpy="0 0 0" xyz="0 0.05 -0.085"/>
         <axis xyz="0 0.707106 -0.707106"/>
@@ -21,5 +21,5 @@
         <parent link="LHipYaw"/>
         <child link="LHip"/>
-        <limit effort="${201.3*68/1000.0}" lower="-0.379472" upper="0.790477" velocity="3.0"/>
+        <limit effort="${effort_type1*speed_red_type1A}" lower="-0.379472" upper="0.790477" velocity="3.0"/>
         <origin rpy="0 0 0" xyz="0 0 0"/>
         <axis xyz="1 0 0"/>
@@ -37,5 +37,5 @@
         <parent link="LHip"/>
         <child link="LHipDummy"/>
-        <limit effort="${130.85*68/1000.0}" lower="-1.535889" upper="0.484090" velocity="3.0"/>
+        <limit effort="${effort_type1*speed_red_type1B}" lower="-1.535889" upper="0.484090" velocity="3.0"/>
         <origin rpy="0 0 0" xyz="0 0 0"/>
         <axis xyz="0 1 0"/>
@@ -53,5 +53,5 @@
         <parent link="LHipDummy"/>
         <child link="LKnee"/>
-        <limit effort="${130.85*68/1000.0}" lower="-0.092346" upper="2.112528" velocity="3.0"/>
+        <limit effort="${effort_type1*speed_red_type1B}" lower="-0.092346" upper="2.112528" velocity="3.0"/>
         <origin rpy="0 0 0" xyz="0 0 -0.1"/>
         <axis xyz="0 1 0"/>
@@ -69,5 +69,5 @@
         <parent link="LKnee"/>
         <child link="l_ankle"/>
-        <limit effort="${130.85*68/1000.0}" lower="-1.189516" upper="0.922747" velocity="3.0"/>
+        <limit effort="${effort_type1*speed_red_type1B}" lower="-1.189516" upper="0.922747" velocity="3.0"/>
         <origin rpy="0 0 0" xyz="0 0 -0.1029"/>
         <axis xyz="0 1 0"/>
@@ -85,5 +85,5 @@
         <parent link="l_ankle"/>
         <child link="l_sole"/>
-        <limit effort="${201.3*68/1000.0}" lower="-0.397880" upper="0.769001" velocity="3.0"/>
+        <limit effort="${effort_type1*speed_red_type1A}" lower="-0.397880" upper="0.769001" velocity="3.0"/>
         <origin rpy="0 0 0" xyz="0 0 0"/>
         <axis xyz="1 0 0"/>
@@ -102,5 +102,5 @@
         <parent link="base_link"/>
         <child link="RHipYaw"/>
-        <limit effort="${201.3*68/1000.0}" lower="-1.145303" upper="0.740810" velocity="3.0"/>
+        <limit effort="${effort_type1*speed_red_type1A}" lower="-1.145303" upper="0.740810" velocity="3.0"/>
         <origin rpy="0 0 0" xyz="0 -0.05 -0.085"/>
         <axis xyz="0 0.707106 0.707106"/>
@@ -119,5 +119,5 @@
         <parent link="RHipYaw"/>
         <child link="RHip"/>
-        <limit effort="${201.3*68/1000.0}" lower="-0.790477" upper="0.379472" velocity="3.0"/>
+        <limit effort="${effort_type1*speed_red_type1A}" lower="-0.790477" upper="0.379472" velocity="3.0"/>
         <origin rpy="0 0 0" xyz="0 0 0"/>
         <axis xyz="1 0 0"/>
@@ -135,5 +135,5 @@
         <parent link="RHip"/>
         <child link="RHipDummy"/>
-        <limit effort="${130.85*68/1000.0}" lower="-1.535889" upper="0.484090" velocity="3.0"/>
+        <limit effort="${effort_type1*speed_red_type1B}" lower="-1.535889" upper="0.484090" velocity="3.0"/>
         <origin rpy="0 0 0" xyz="0 0 0"/>
         <axis xyz="0 1 0"/>
@@ -151,5 +151,5 @@
         <parent link="RHipDummy"/>
         <child link="RKnee"/>
-        <limit effort="${130.85*68/1000.0}" lower="-0.103083" upper="2.120198" velocity="3.0"/>
+        <limit effort="${effort_type1*speed_red_type1B}" lower="-0.103083" upper="2.120198" velocity="3.0"/>
         <origin rpy="0 0 0" xyz="0 0 -0.1"/>
         <axis xyz="0 1 0"/>
@@ -167,5 +167,5 @@
         <parent link="RKnee"/>
         <child link="r_ankle"/>
-        <limit effort="${130.85*68/1000.0}" lower="-1.186448" upper="0.932056" velocity="3.0"/>
+        <limit effort="${effort_type1*speed_red_type1B}" lower="-1.186448" upper="0.932056" velocity="3.0"/>
         <origin rpy="0 0 0" xyz="0 0 -0.1029"/>
         <axis xyz="0 1 0"/>
@@ -183,5 +183,5 @@
         <parent link="r_ankle"/>
         <child link="r_sole"/>
-        <limit effort="${201.3*68/1000.0}" lower="-0.768992" upper="0.397935" velocity="3.0"/>
+        <limit effort="${effort_type1*speed_red_type1A}" lower="-0.768992" upper="0.397935" velocity="3.0"/>
         <origin rpy="0 0 0" xyz="0 0 0"/>
         <axis xyz="1 0 0"/>

File: nao_dcm_common/nao_dcm_description/urdf/modules/robot.xacro (robot description, xacro)
@@ -10,4 +10,13 @@
 	<xacro:property name="use_odroid" value="true" />
 	<xacro:property name="use_hector_imu" value="false" />
+	<xacro:property name="effort_type1" value="0.0161" />
+	<xacro:property name="effort_type2" value="0.0049" />
+	<xacro:property name="effort_type3" value="0.0062" />
+	<xacro:property name="speed_red_type1A" value="201.3" />
+	<xacro:property name="speed_red_type1B" value="130.85" />
+	<xacro:property name="speed_red_type2A" value="50.61" />
+	<xacro:property name="speed_red_type2B" value="36.24" />
+	<xacro:property name="speed_red_type3A" value="150.27" />
+	<xacro:property name="speed_red_type3B" value="173.22" />
 	<!-- Which IMU plugin to use (hector or default) -->
 	<xacro:if value="${use_hector_imu}">

File: nao_dcm_common/nao_dcm_description/urdf/nao_dcm_H21_control.xacro (robot description, xacro)
@@ -8,5 +8,5 @@
 			<!-- Dummy Values -->
 			<hardwareInterface>PositionJointInterface</hardwareInterface>
-			<mechanicalReduction>150.27</mechanicalReduction>
+			<mechanicalReduction>${speed_red_type3A}</mechanicalReduction>
 		</actuator>
 	</transmission>
@@ -17,5 +17,5 @@
 			<!-- Dummy Values -->
 			<hardwareInterface>PositionJointInterface</hardwareInterface>
-			<mechanicalReduction>173.22</mechanicalReduction>
+			<mechanicalReduction>${speed_red_type3B}</mechanicalReduction>
 		</actuator>
 	</transmission>
@@ -29,5 +29,5 @@
 				<!-- Dummy Values -->
 				<hardwareInterface>PositionJointInterface</hardwareInterface>
-				<mechanicalReduction>150.27</mechanicalReduction>
+				<mechanicalReduction>${speed_red_type3A}</mechanicalReduction>
 			</actuator>
 		</transmission>
@@ -38,5 +38,5 @@
 				<!-- Dummy Values -->
 				<hardwareInterface>PositionJointInterface</hardwareInterface>
-				<mechanicalReduction>150.27</mechanicalReduction>
+				<mechanicalReduction>${speed_red_type3A}</mechanicalReduction>
 			</actuator>
 		</transmission>
@@ -47,5 +47,5 @@
 				<!-- Dummy Values -->
 				<hardwareInterface>PositionJointInterface</hardwareInterface>
-				<mechanicalReduction>173.22</mechanicalReduction>
+				<mechanicalReduction>${speed_red_type3B}</mechanicalReduction>
 			</actuator>
 		</transmission>
@@ -56,5 +56,5 @@
 				<!-- Dummy Values -->
 				<hardwareInterface>PositionJointInterface</hardwareInterface>
-				<mechanicalReduction>173.22</mechanicalReduction>
+				<mechanicalReduction>${speed_red_type3B}</mechanicalReduction>
 			</actuator>
 		</transmission>
@@ -71,5 +71,5 @@
 				<!-- Dummy Values -->
 				<hardwareInterface>PositionJointInterface</hardwareInterface>
-				<mechanicalReduction>201.3</mechanicalReduction>
+				<mechanicalReduction>${speed_red_type1A}</mechanicalReduction>
 			</actuator>
 		</transmission>
@@ -80,5 +80,5 @@
 				<!-- Dummy Values -->
 				<hardwareInterface>PositionJointInterface</hardwareInterface>
-				<mechanicalReduction>201.3</mechanicalReduction>
+				<mechanicalReduction>${speed_red_type1A}</mechanicalReduction>
 			</actuator>
 		</transmission>
@@ -89,5 +89,5 @@
 				<!-- Dummy Values -->
 				<hardwareInterface>PositionJointInterface</hardwareInterface>
-				<mechanicalReduction>130.85</mechanicalReduction>
+				<mechanicalReduction>${speed_red_type1B}</mechanicalReduction>
 			</actuator>
 		</transmission>
@@ -98,5 +98,5 @@
 				<!-- Dummy Values -->
 				<hardwareInterface>PositionJointInterface</hardwareInterface>
-				<mechanicalReduction>130.85</mechanicalReduction>
+				<mechanicalReduction>${speed_red_type1B}</mechanicalReduction>
 			</actuator>
 		</transmission>
@@ -107,5 +107,5 @@
 				<!-- Dummy Values -->
 				<hardwareInterface>PositionJointInterface</hardwareInterface>
-				<mechanicalReduction>130.85</mechanicalReduction>
+				<mechanicalReduction>${speed_red_type1B}</mechanicalReduction>
 			</actuator>
 		</transmission>
@@ -116,5 +116,5 @@
 				<!-- Dummy Values -->
 				<hardwareInterface>PositionJointInterface</hardwareInterface>
-				<mechanicalReduction>201.3</mechanicalReduction>
+				<mechanicalReduction>${speed_red_type1A}</mechanicalReduction>
 			</actuator>
 		</transmission>

File: nao_dcm_common/nao_dcm_description/urdf/nao_dcm_H25_control.xacro (robot description, xacro)
@@ -8,5 +8,5 @@
 			<!-- Dummy Values -->
 			<hardwareInterface>PositionJointInterface</hardwareInterface>
-			<mechanicalReduction>150.27</mechanicalReduction>
+			<mechanicalReduction>${speed_red_type3A}</mechanicalReduction>
 		</actuator>
 	</transmission>
@@ -17,5 +17,5 @@
 			<!-- Dummy Values -->
 			<hardwareInterface>PositionJointInterface</hardwareInterface>
-			<mechanicalReduction>173.22</mechanicalReduction>
+			<mechanicalReduction>${speed_red_type3B}</mechanicalReduction>
 		</actuator>
 	</transmission>
@@ -29,5 +29,5 @@
 				<!-- Dummy Values -->
 				<hardwareInterface>PositionJointInterface</hardwareInterface>
-				<mechanicalReduction>150.27</mechanicalReduction>
+				<mechanicalReduction>${speed_red_type3A}</mechanicalReduction>
 			</actuator>
 		</transmission>
@@ -38,5 +38,5 @@
 				<!-- Dummy Values -->
 				<hardwareInterface>PositionJointInterface</hardwareInterface>
-				<mechanicalReduction>150.27</mechanicalReduction>
+				<mechanicalReduction>${speed_red_type3A}</mechanicalReduction>
 			</actuator>
 		</transmission>
@@ -47,5 +47,5 @@
 				<!-- Dummy Values -->
 				<hardwareInterface>PositionJointInterface</hardwareInterface>
-				<mechanicalReduction>50.61</mechanicalReduction>
+				<mechanicalReduction>${speed_red_type2A}</mechanicalReduction>
 			</actuator>
 		</transmission>
@@ -56,5 +56,5 @@
 				<!-- Dummy Values -->
 				<hardwareInterface>PositionJointInterface</hardwareInterface>
-				<mechanicalReduction>36.24</mechanicalReduction>
+				<mechanicalReduction>${speed_red_type2B}</mechanicalReduction>
 			</actuator>
 		</transmission>
@@ -65,5 +65,5 @@
 				<!-- Dummy Values -->
 				<hardwareInterface>PositionJointInterface</hardwareInterface>
-				<mechanicalReduction>173.22</mechanicalReduction>
+				<mechanicalReduction>${speed_red_type3B}</mechanicalReduction>
 			</actuator>
 		</transmission>
@@ -74,5 +74,5 @@
 				<!-- Dummy Values -->
 				<hardwareInterface>PositionJointInterface</hardwareInterface>
-				<mechanicalReduction>173.22</mechanicalReduction>
+				<mechanicalReduction>${speed_red_type3B}</mechanicalReduction>
 			</actuator>
 		</transmission>
@@ -89,5 +89,5 @@
 				<!-- Dummy Values -->
 				<hardwareInterface>PositionJointInterface</hardwareInterface>
-				<mechanicalReduction>201.3</mechanicalReduction>
+				<mechanicalReduction>${speed_red_type1A}</mechanicalReduction>
 			</actuator>
 		</transmission>
@@ -98,5 +98,5 @@
 				<!-- Dummy Values -->
 				<hardwareInterface>PositionJointInterface</hardwareInterface>
-				<mechanicalReduction>201.3</mechanicalReduction>
+				<mechanicalReduction>${speed_red_type1A}</mechanicalReduction>
 			</actuator>
 		</transmission>
@@ -107,5 +107,5 @@
 				<!-- Dummy Values -->
 				<hardwareInterface>PositionJointInterface</hardwareInterface>
-				<mechanicalReduction>130.85</mechanicalReduction>
+				<mechanicalReduction>${speed_red_type1B}</mechanicalReduction>
 			</actuator>
 		</transmission>
@@ -116,5 +116,5 @@
 				<!-- Dummy Values -->
 				<hardwareInterface>PositionJointInterface</hardwareInterface>
-				<mechanicalReduction>130.85</mechanicalReduction>
+				<mechanicalReduction>${speed_red_type1B}</mechanicalReduction>
 			</actuator>
 		</transmission>
@@ -125,5 +125,5 @@
 				<!-- Dummy Values -->
 				<hardwareInterface>PositionJointInterface</hardwareInterface>
-				<mechanicalReduction>130.85</mechanicalReduction>
+				<mechanicalReduction>${speed_red_type1B}</mechanicalReduction>
 			</actuator>
 		</transmission>
@@ -134,5 +134,5 @@
 				<!-- Dummy Values -->
 				<hardwareInterface>PositionJointInterface</hardwareInterface>
-				<mechanicalReduction>201.3</mechanicalReduction>
+				<mechanicalReduction>${speed_red_type1A}</mechanicalReduction>
 			</actuator>
 		</transmission>

File: nao_dcm_common/nao_dcm_description/urdf/nao_dcm_gazebo.xacro (robot description, xacro)
@@ -1,4 +1,34 @@
 <?xml version="1.0"?>
 <robot xmlns:xacro="http://www.ros.org/wiki/xacro">
+    <!-- MACROS FOR DISABLE LINKS -->
+    <xacro:macro name="DisabledLinks" params="side side_small">
+        <plugin name="${side}Finger11" filename="libgazebo_disable_link_plugin.so">
+            <link>${side}Finger11</link>
+        </plugin>
+        <plugin name="${side}Finger12" filename="libgazebo_disable_link_plugin.so">
+            <link>${side}Finger12</link>
+        </plugin>
+        <plugin name="${side}Finger13" filename="libgazebo_disable_link_plugin.so">
+            <link>${side}Finger13</link>
+        </plugin>
+        <plugin name="${side}Finger21" filename="libgazebo_disable_link_plugin.so">
+            <link>${side}Finger21</link>
+        </plugin>
+        <plugin name="${side}Finger22" filename="libgazebo_disable_link_plugin.so">
+            <link>${side}Finger22</link>
+        </plugin>
+        <plugin name="${side}Finger23" filename="libgazebo_disable_link_plugin.so">
+            <link>${side}Finger23</link>
+        </plugin>
+        <plugin name="${side}Thumb1" filename="libgazebo_disable_link_plugin.so">
+            <link>${side}Thumb1</link>
+        </plugin>
+        <plugin name="${side}Thumb2" filename="libgazebo_disable_link_plugin.so">
+            <link>${side}Thumb2</link>
+        </plugin>
+        <plugin name="${side_small}_gripper" filename="libgazebo_disable_link_plugin.so">
+            <link>${side_small}_gripper</link>
+        </plugin>
+    </xacro:macro>
     <!-- MACROS FOR MIMIC JOINTS -->
     <!-- Fingers -->
@@ -71,4 +101,6 @@
         <xacro:ThumbMimics side="L"/>
         <xacro:ThumbMimics side="R"/>
+        <xacro:DisabledLinks side="L" side_small="l"/>
+        <xacro:DisabledLinks side="R" side_small="r"/>
     </gazebo>
     <!-- END OF GAZEBO ROS CONTROL PLUGIN -->
