Commit message: Small tweaking of the PIDs..Added Xtion helmet.

File: nao_dcm_common/nao_dcm_description/urdf/modules/robot.xacro (robot description, xacro)
@@ -6,6 +6,7 @@
 	<xacro:property name="scale" value="0.001" />
 	<xacro:property name="nao_meshes" value="true" />
-	<xacro:property name="use_helmet" value="true" />
+	<xacro:property name="use_helmet" value="false" />
 	<xacro:property name="helmet_cameras_viz" value="false" />
+	<xacro:property name="use_xtion" value="true" />
 	<xacro:property name="use_odroid" value="true" />
 	<xacro:property name="use_hector_imu" value="false" />
@@ -42,4 +43,8 @@
 		<xacro:include filename="$(find nao_dcm_description)/urdf/modules/helmet_cameras.xacro" />
 	</xacro:if>
+	<!-- Whether to use Nao helmet with ASUS Xtion or not -->
+	<xacro:if value="${use_xtion}">
+		<xacro:include filename="$(find nao_dcm_description)/urdf/modules/helmet_xtion.xacro" />
+	</xacro:if>
 	<!-- Whether to use Odroid or not -->
 	<xacro:if value="${use_odroid}">

File: nao_dcm_common/nao_dcm_description/urdf/nao_dcm_gazebo.xacro (robot description, xacro)
@@ -94,5 +94,4 @@
             <multiplier>1.0</multiplier>
             <offset>0.0</offset>
-            <sensitiveness>0.1</sensitiveness>
         </plugin>
         <xacro:FingerMimics side="L" num="1"/>
