Commit message: Cleaned URDF and MoveIt! config

File: nao_dcm_common/nao_dcm_description/urdf/modules/helmet.xacro (robot description, xacro)
@@ -1,4 +1,21 @@
 <?xml version="1.0"?>
 <robot xmlns:xacro="http://www.ros.org/wiki/xacro">
+	<!-- XACRO MACROS FOR VISUALS AND COLLISIONS -->
+	<xacro:macro name="visuals_collisions_helmet" params="">
+		<visual>
+			<origin xyz="0 0 0" rpy="0 -0 0"/>
+			<geometry>
+				<mesh filename="package://nao_dcm_description/meshes/helmet.dae"  scale="${scale} ${scale} ${scale}"/>
+			</geometry>
+			<material name="LightGrey"/>
+		</visual>
+		<!-- <collision>
+			<origin xyz="0 0 0" rpy="0 -0 0"/>
+			<geometry>
+				<mesh filename="package://nao_dcm_description/meshes/helmet.dae"  scale="${scale} ${scale} ${scale}"/>
+			</geometry>
+			<material name="LightGrey"/>
+		</collision> -->
+	</xacro:macro>
 	<joint name="head-helmet" type="fixed">
         <parent link="gaze"/>

File: nao_dcm_common/nao_dcm_description/urdf/modules/helmet_xtion.xacro (robot description, xacro)
@@ -1,7 +1,7 @@
 <?xml version="1.0"?>
 <robot xmlns:xacro="http://www.ros.org/wiki/xacro">
-	<!-- XACRO MACROS FOR VISUALS AND COLLISIONS -->
-    <xacro:macro name="visuals_collisions_helmet_xtion" params="">
-    	<visual>
+  <!-- XACRO MACROS FOR VISUALS AND COLLISIONS -->
+  <xacro:macro name="visuals_collisions_helmet_xtion" params="">
+    <visual>
 			<origin xyz="0 0 0" rpy="0 0 0"/>
 			<geometry>
@@ -11,7 +11,8 @@
 		</visual>
 		<collision>
-			<origin xyz="0 0 0" rpy="0 0 0"/>
+			<origin xyz="0 0 0.05" rpy="${PI_2} 0 0"/>
 			<geometry>
-				<mesh filename="package://nao_dcm_description/meshes/helmet_xtion.dae"/>
+				<!-- <mesh filename="package://nao_dcm_description/meshes/helmet_xtion.dae"/> -->
+        <cylinder radius="0.01" length="0.14"/>
 			</geometry>
 			<material name="LightGrey"/>
@@ -33,39 +34,41 @@
     <link name="xtion"/>
     <!-- GAZEBO SPECIFIC FOR XTION -->
-    <gazebo reference="helmet-xtion">
-    	<sensor type="depth" name="xtion">
-        <always_on>true</always_on>
-        <update_rate>30.0</update_rate>
-        <camera>
-          <horizontal_fov>${60.0*PI/180.0}</horizontal_fov>
-          <image>
-            <format>R8G8B8</format>
-            <width>640</width>
-            <height>480</height>
-          </image>
-          <clip>
-            <near>0.05</near>
-            <far>8.0</far>
-          </clip>
-        </camera>
-        <plugin name="xtion_camera_controller" filename="libgazebo_ros_openni_kinect.so">
-          <cameraName>xtion</cameraName>
-          <alwaysOn>true</alwaysOn>
-          <updateRate>30</updateRate>
-          <imageTopicName>xtion/rgb/image_raw</imageTopicName>
-          <depthImageTopicName>xtion/depth/image_raw</depthImageTopicName>
-          <pointCloudTopicName>xtion/depth/points</pointCloudTopicName>
-          <cameraInfoTopicName>xtion/rgb/camera_info</cameraInfoTopicName>
-          <depthImageCameraInfoTopicName>xtion/depth/camera_info</depthImageCameraInfoTopicName>
-          <frameName>xtion</frameName>
-          <baseline>0.1</baseline>
-          <distortion_k1>0.0</distortion_k1>
-          <distortion_k2>0.0</distortion_k2>
-          <distortion_k3>0.0</distortion_k3>
-          <distortion_t1>0.0</distortion_t1>
-          <distortion_t2>0.0</distortion_t2>
-          <pointCloudCutoff>0.4</pointCloudCutoff>
-        </plugin>
-      </sensor>
-	</gazebo>
+    <xacro:if value="${use_gazebo}">
+      <gazebo reference="helmet-xtion">
+      	<sensor type="depth" name="xtion">
+          <always_on>true</always_on>
+          <update_rate>30.0</update_rate>
+          <camera>
+            <horizontal_fov>${60.0*PI/180.0}</horizontal_fov>
+            <image>
+              <format>R8G8B8</format>
+              <width>640</width>
+              <height>480</height>
+            </image>
+            <clip>
+              <near>0.05</near>
+              <far>8.0</far>
+            </clip>
+          </camera>
+          <plugin name="xtion_camera_controller" filename="libgazebo_ros_openni_kinect.so">
+            <cameraName>xtion</cameraName>
+            <alwaysOn>true</alwaysOn>
+            <updateRate>30</updateRate>
+            <imageTopicName>xtion/rgb/image_raw</imageTopicName>
+            <depthImageTopicName>xtion/depth/image_raw</depthImageTopicName>
+            <pointCloudTopicName>xtion/depth/points</pointCloudTopicName>
+            <cameraInfoTopicName>xtion/rgb/camera_info</cameraInfoTopicName>
+            <depthImageCameraInfoTopicName>xtion/depth/camera_info</depthImageCameraInfoTopicName>
+            <frameName>xtion</frameName>
+            <baseline>0.1</baseline>
+            <distortion_k1>0.0</distortion_k1>
+            <distortion_k2>0.0</distortion_k2>
+            <distortion_k3>0.0</distortion_k3>
+            <distortion_t1>0.0</distortion_t1>
+            <distortion_t2>0.0</distortion_t2>
+            <pointCloudCutoff>0.4</pointCloudCutoff>
+          </plugin>
+        </sensor>
+  	</gazebo>
+  </xacro:if>
 </robot>

File: nao_dcm_common/nao_dcm_description/urdf/modules/odroid_bag.xacro (robot description, xacro)
@@ -11,7 +11,8 @@
 		</visual>
 		<collision>
-			<origin xyz="0 0 0" rpy="0 0 0"/>
+			<origin xyz="-0.02 0 0" rpy="0 0 0"/>
 			<geometry>
-				<mesh filename="package://nao_dcm_description/meshes/odroid_bag.dae"  scale="${scale} ${scale} ${scale}"/>
+				<!-- <mesh filename="package://nao_dcm_description/meshes/odroid_bag.dae"  scale="${scale} ${scale} ${scale}"/> -->
+				<box size="0.01 0.01 0.01"/>
 			</geometry>
 			<material name="LightGrey"/>
@@ -27,7 +28,8 @@
 		</visual>
 		<collision>
-			<origin xyz="0 0 0" rpy="0 0 0"/>
+			<origin xyz="0 0.01 0" rpy="0 0 0"/>
 			<geometry>
-				<mesh filename="package://nao_dcm_description/meshes/odroid.dae"  scale="${scale} ${scale} ${scale}"/>
+				<!-- <mesh filename="package://nao_dcm_description/meshes/odroid.dae"  scale="${scale} ${scale} ${scale}"/> -->
+				<box size="0.01 0.01 0.01"/>
 			</geometry>
 			<material name="LightGrey"/>

File: nao_dcm_common/nao_dcm_description/urdf/modules/robot.xacro (robot description, xacro)
@@ -11,4 +11,5 @@
 	<xacro:property name="use_odroid" value="true" />
 	<xacro:property name="use_hector_imu" value="false" />
+	<xacro:property name="use_gazebo" value="true" />
 	<xacro:property name="effort_type1" value="0.0161" />
 	<xacro:property name="effort_type2" value="0.0049" />
@@ -28,5 +29,7 @@
 	</xacro:unless>
 	<xacro:include filename="$(find nao_dcm_description)/urdf/nao_dcm_visuals_collisions.xacro" />
-	<xacro:include filename="$(find nao_dcm_description)/urdf/nao_dcm_gazebo.xacro" />
+	<xacro:if value="${use_gazebo}">
+		<xacro:include filename="$(find nao_dcm_description)/urdf/nao_dcm_gazebo.xacro" />
+	</xacro:if>
 	<!-- Load xacro modules/parts of the robot -->
 	<xacro:include filename="$(find nao_dcm_description)/urdf/modules/torso.xacro" />

File: nao_dcm_common/nao_dcm_description/urdf/nao_dcm_visuals_collisions.xacro (robot description, xacro)
@@ -19,20 +19,4 @@
     <!-- END OF MATERIALS -->
     <!-- XACRO MACROS FOR VISUALS AND COLLISIONS -->
-    <xacro:macro name="visuals_collisions_helmet" params="">
-		<visual>
-			<origin xyz="0 0 0" rpy="0 -0 0"/>
-			<geometry>
-				<mesh filename="package://nao_dcm_description/meshes/helmet.dae"  scale="${scale} ${scale} ${scale}"/>
-			</geometry>
-			<material name="LightGrey"/>
-		</visual>
-		<collision>
-			<origin xyz="0 0 0" rpy="0 -0 0"/>
-			<geometry>
-				<mesh filename="package://nao_dcm_description/meshes/helmet.dae"  scale="${scale} ${scale} ${scale}"/>
-			</geometry>
-			<material name="LightGrey"/>
-		</collision>
-	</xacro:macro>
 	<xacro:macro name="visuals_collisions_torso" params="">
 		<xacro:unless value="${nao_meshes}">
